File: hardware/udriver3/OMODRI_CAN.sch (KiCad schematic (older format))
At the start: 4 parts

Commit message: Update of the BOM. Not yet finished.
Parts:
- C110: renamed from C?; footprint (none) -> Capacitor_SMD:C_0201_0603Metric; DigiKey (none) -> 490-14450-1-ND; Farnell (none) -> 2990681; Mouser (none) -> 81-GRM033C71A104KE4D; Part No (none) -> GRM033C71A104KE14D; RS (none) -> 185-1751; Rated Voltage (none) -> 10V; Rated voltage 10V -> (none)
- gave numbers to parts that had none: 3
Changed lines of the file:
@@
 $Descr A4 11693 8268
 encoding utf-8
-Sheet 6 7
+Sheet 6 8
 Title "Open MOtor DRiver Initiative (OMODRI)"
 Date ""
@@
 $EndDescr
 $Comp
-L Interface_CAN_LIN:TCAN332G U?
+L Interface_CAN_LIN:TCAN332G U9
 U 1 1 60EC8ED3
 P 5300 3650
-F 0 "U?" H 5400 4100 50  0000 C CNN
+F 0 "U9" H 5400 4100 50  0000 C CNN
 F 1 "TCAN332G" H 5550 4000 50  0000 C CNN
 F 2 "" H 5300 3150 50  0001 C CIN
@@
 AR Path="/5F387075/60ECB2D3" Ref="C?"  Part="1"
 AR Path="/60E4937F/60ECB2D3" Ref="C?"  Part="1"
-AR Path="/60EC8491/60ECB2D3" Ref="C?"  Part="1"
-F 0 "C?" H 5050 3000 50  0000 L CNN
+AR Path="/60EC8491/60ECB2D3" Ref="C110"  Part="1"
+F 0 "C110" H 5050 3000 50  0000 L CNN
 F 1 "100nF" H 5050 2900 50  0000 L CNN
-F 2 "" H 4988 2750 50  0001 C CNN
-F 3 "~" H 4950 2900 50  0001 C CNN
-F 4 "10V" H 4950 2900 50  0001 C CNN "Rated voltage"
+F 2 "Capacitor_SMD:C_0201_0603Metric" H 4988 2750 50  0001 C CNN
+F 3 "https://www.murata.com/en-eu/products/productdetail?partno=GRM033C71A104KE14%23" H 4950 2900 50  0001 C CNN
+F 4 "" H 4950 2900 50  0001 C CNN "Rated voltage"
+F 5 "490-14450-1-ND" H 4950 2900 50  0001 C CNN "DigiKey"
+F 6 "2990681" H 4950 2900 50  0001 C CNN "Farnell"
+F 7 "81-GRM033C71A104KE4D" H 4950 2900 50  0001 C CNN "Mouser"
+F 8 "GRM033C71A104KE14D" H 4950 2900 50  0001 C CNN "Part No"
+F 9 "185-1751" H 4950 2900 50  0001 C CNN "RS"
+F 10 "10V" H 4950 2900 50  0001 C CNN "Rated Voltage"
 	1    4950 2900
 	1    0    0    -1
@@
 AR Path="/5F387075/60ECB2D9" Ref="#PWR?"  Part="1"
 AR Path="/60E4937F/60ECB2D9" Ref="#PWR?"  Part="1"
-AR Path="/60EC8491/60ECB2D9" Ref="#PWR0129"  Part="1"
-F 0 "#PWR0129" H 4950 2850 50  0001 C CNN
+AR Path="/60EC8491/60ECB2D9" Ref="#PWR080"  Part="1"
+F 0 "#PWR080" H 4950 2850 50  0001 C CNN
 F 1 "GND" H 4955 2927 50  0000 C CNN
 F 2 "" H 4950 3100 50  0001 C CNN
@@
 AR Path="/5F387075/60ECB715" Ref="#PWR?"  Part="1"
 AR Path="/60E4937F/60ECB715" Ref="#PWR?"  Part="1"
-AR Path="/60EC8491/60ECB715" Ref="#PWR0130"  Part="1"
-F 0 "#PWR0130" H 5300 3850 50  0001 C CNN
+AR Path="/60EC8491/60ECB715" Ref="#PWR081"  Part="1"
+F 0 "#PWR081" H 5300 3850 50  0001 C CNN
 F 1 "GND" H 5305 3927 50  0000 C CNN
 F 2 "" H 5300 4100 50  0001 C CNN
@@
 AR Path="/5F387075/60ED7D95" Ref="R?"  Part="1"
 AR Path="/60E4937F/60ED7D95" Ref="R?"  Part="1"
-AR Path="/60EC8491/60ED7D95" Ref="R?"  Part="1"
-F 0 "R?" H 6270 3696 50  0000 L CNN
+AR Path="/60EC8491/60ED7D95" Ref="R42"  Part="1"
+F 0 "R42" H 6270 3696 50  0000 L CNN
 F 1 "120" H 6270 3605 50  0000 L CNN
 F 2 "" V 6130 3650 50  0001 C CNN
@@
 	5850 3500 6200 3500
 $Comp
-L Connector_Generic:Conn_01x02 J?
+L Connector_Generic:Conn_01x02 J5
 U 1 1 60EDAE2F
 P 6800 3600
-F 0 "J?" H 6880 3592 50  0000 L CNN
+F 0 "J5" H 6880 3592 50  0000 L CNN
 F 1 "Conn_01x02" H 6880 3501 50  0000 L CNN
 F 2 "" H 6800 3600 50  0001 C CNN

Commit message: Power supply distribution updated.
Parts:
- R45: renamed from R42; footprint (none) -> Resistor_SMD:R_0201_0603Metric; DigiKey (none) -> P122692CT-ND; Farnell (none) -> 2396857; Mouser (none) -> 667-ERJ-1GNF1200C; Part No (none) -> ERJ-1GNF1200C
- renumbered C110 to C107
Changed lines of the file:
@@
 AR Path="/5F387075/60ECB2D3" Ref="C?"  Part="1"
 AR Path="/60E4937F/60ECB2D3" Ref="C?"  Part="1"
-AR Path="/60EC8491/60ECB2D3" Ref="C110"  Part="1"
-F 0 "C110" H 5050 3000 50  0000 L CNN
+AR Path="/60EC8491/60ECB2D3" Ref="C107"  Part="1"
+F 0 "C107" H 5050 3000 50  0000 L CNN
 F 1 "100nF" H 5050 2900 50  0000 L CNN
 F 2 "Capacitor_SMD:C_0201_0603Metric" H 4988 2750 50  0001 C CNN
@@
 AR Path="/5F387075/60ECB2D9" Ref="#PWR?"  Part="1"
 AR Path="/60E4937F/60ECB2D9" Ref="#PWR?"  Part="1"
-AR Path="/60EC8491/60ECB2D9" Ref="#PWR080"  Part="1"
-F 0 "#PWR080" H 4950 2850 50  0001 C CNN
+AR Path="/60EC8491/60ECB2D9" Ref="#PWR084"  Part="1"
+F 0 "#PWR084" H 4950 2850 50  0001 C CNN
 F 1 "GND" H 4955 2927 50  0000 C CNN
 F 2 "" H 4950 3100 50  0001 C CNN
@@
 AR Path="/5F387075/60ECB715" Ref="#PWR?"  Part="1"
 AR Path="/60E4937F/60ECB715" Ref="#PWR?"  Part="1"
-AR Path="/60EC8491/60ECB715" Ref="#PWR081"  Part="1"
-F 0 "#PWR081" H 5300 3850 50  0001 C CNN
+AR Path="/60EC8491/60ECB715" Ref="#PWR085"  Part="1"
+F 0 "#PWR085" H 5300 3850 50  0001 C CNN
 F 1 "GND" H 5305 3927 50  0000 C CNN
 F 2 "" H 5300 4100 50  0001 C CNN
@@
 AR Path="/5F387075/60ED7D95" Ref="R?"  Part="1"
 AR Path="/60E4937F/60ED7D95" Ref="R?"  Part="1"
-AR Path="/60EC8491/60ED7D95" Ref="R42"  Part="1"
-F 0 "R42" H 6270 3696 50  0000 L CNN
+AR Path="/60EC8491/60ED7D95" Ref="R45"  Part="1"
+F 0 "R45" H 6270 3696 50  0000 L CNN
 F 1 "120" H 6270 3605 50  0000 L CNN
-F 2 "" V 6130 3650 50  0001 C CNN
-F 3 "~" H 6200 3650 50  0001 C CNN
+F 2 "Resistor_SMD:R_0201_0603Metric" V 6130 3650 50  0001 C CNN
+F 3 "https://industrial.panasonic.com/cdbs/www-data/pdf/RDA0000/AOA0000C304.pdf" H 6200 3650 50  0001 C CNN
+F 4 "P122692CT-ND" H 6200 3650 50  0001 C CNN "DigiKey"
+F 5 "2396857" H 6200 3650 50  0001 C CNN "Farnell"
+F 6 "667-ERJ-1GNF1200C" H 6200 3650 50  0001 C CNN "Mouser"
+F 7 "ERJ-1GNF1200C" H 6200 3650 50  0001 C CNN "Part No"
 	1    6200 3650
 	1    0    0    -1

Commit message: Updated version with 28388D pin matching PAL design.
Parts:
- renumbered C107 to C131, R45 to R69, U9 to U10
Changed lines of the file:
@@
 $Descr A4 11693 8268
 encoding utf-8
-Sheet 6 8
+Sheet 6 10
 Title "Open MOtor DRiver Initiative (OMODRI)"
 Date ""
@@
 $EndDescr
 $Comp
-L Interface_CAN_LIN:TCAN332G U9
+L Interface_CAN_LIN:TCAN332G U10
 U 1 1 60EC8ED3
 P 5300 3650
-F 0 "U9" H 5400 4100 50  0000 C CNN
+F 0 "U10" H 5400 4100 50  0000 C CNN
 F 1 "TCAN332G" H 5550 4000 50  0000 C CNN
 F 2 "" H 5300 3150 50  0001 C CIN
@@
 AR Path="/5F387075/60ECB2D3" Ref="C?"  Part="1"
 AR Path="/60E4937F/60ECB2D3" Ref="C?"  Part="1"
-AR Path="/60EC8491/60ECB2D3" Ref="C107"  Part="1"
-F 0 "C107" H 5050 3000 50  0000 L CNN
+AR Path="/60EC8491/60ECB2D3" Ref="C131"  Part="1"
+F 0 "C131" H 5050 3000 50  0000 L CNN
 F 1 "100nF" H 5050 2900 50  0000 L CNN
 F 2 "Capacitor_SMD:C_0201_0603Metric" H 4988 2750 50  0001 C CNN
@@
 AR Path="/5F387075/60ECB2D9" Ref="#PWR?"  Part="1"
 AR Path="/60E4937F/60ECB2D9" Ref="#PWR?"  Part="1"
-AR Path="/60EC8491/60ECB2D9" Ref="#PWR084"  Part="1"
-F 0 "#PWR084" H 4950 2850 50  0001 C CNN
+AR Path="/60EC8491/60ECB2D9" Ref="#PWR0110"  Part="1"
+F 0 "#PWR0110" H 4950 2850 50  0001 C CNN
 F 1 "GND" H 4955 2927 50  0000 C CNN
 F 2 "" H 4950 3100 50  0001 C CNN
@@
 AR Path="/5F387075/60ECB715" Ref="#PWR?"  Part="1"
 AR Path="/60E4937F/60ECB715" Ref="#PWR?"  Part="1"
-AR Path="/60EC8491/60ECB715" Ref="#PWR085"  Part="1"
-F 0 "#PWR085" H 5300 3850 50  0001 C CNN
+AR Path="/60EC8491/60ECB715" Ref="#PWR0111"  Part="1"
+F 0 "#PWR0111" H 5300 3850 50  0001 C CNN
 F 1 "GND" H 5305 3927 50  0000 C CNN
 F 2 "" H 5300 4100 50  0001 C CNN
@@
 AR Path="/5F387075/60ED7D95" Ref="R?"  Part="1"
 AR Path="/60E4937F/60ED7D95" Ref="R?"  Part="1"
-AR Path="/60EC8491/60ED7D95" Ref="R45"  Part="1"
-F 0 "R45" H 6270 3696 50  0000 L CNN
+AR Path="/60EC8491/60ED7D95" Ref="R69"  Part="1"
+F 0 "R69" H 6270 3696 50  0000 L CNN
 F 1 "120" H 6270 3605 50  0000 L CNN
 F 2 "Resistor_SMD:R_0201_0603Metric" V 6130 3650 50  0001 C CNN

Commit message: All footprints are present. DRV with 2 power branches.
Parts:
- J10: renamed from J5; footprint (none) -> Connector_Hirose:Hirose_DF13-02P-1.25DSA_1x02_P1.25mm_Vertical
- U10: footprint (none) -> Package_TO_SOT_SMD:TSOT-23-8; DigiKey (none) -> 296-48677-1-ND; Farnell (none) -> 3009409; Mouser (none) -> 595-TCAN332GDCNR; Part No (none) -> TCAN332GDCNR
- renumbered C131 to C141, R69 to R67
Connections:
- net 3V3 renamed VDD_3V3
Changed lines of the file:
@@
 F 0 "U10" H 5400 4100 50  0000 C CNN
 F 1 "TCAN332G" H 5550 4000 50  0000 C CNN
-F 2 "" H 5300 3150 50  0001 C CIN
+F 2 "Package_TO_SOT_SMD:TSOT-23-8" H 5300 3150 50  0001 C CIN
 F 3 "https://www.ti.com/lit/ds/symlink/tcan330g.pdf" H 5300 3650 50  0001 C CNN
+F 4 "296-48677-1-ND" H 5300 3650 50  0001 C CNN "DigiKey"
+F 5 "3009409" H 5300 3650 50  0001 C CNN "Farnell"
+F 6 "595-TCAN332GDCNR" H 5300 3650 50  0001 C CNN "Mouser"
+F 7 "TCAN332GDCNR" H 5300 3650 50  0001 C CNN "Part No"
 	1    5300 3650
 	1    0    0    -1
 $EndComp
 Text GLabel 4850 2750 0    50   Input ~ 0
-3V3
+VDD_3V3
 $Comp
 L Device:C C?
@@
 AR Path="/5F387075/60ECB2D3" Ref="C?"  Part="1"
 AR Path="/60E4937F/60ECB2D3" Ref="C?"  Part="1"
-AR Path="/60EC8491/60ECB2D3" Ref="C131"  Part="1"
-F 0 "C131" H 5050 3000 50  0000 L CNN
+AR Path="/60EC8491/60ECB2D3" Ref="C141"  Part="1"
+F 0 "C141" H 5050 3000 50  0000 L CNN
 F 1 "100nF" H 5050 2900 50  0000 L CNN
 F 2 "Capacitor_SMD:C_0201_0603Metric" H 4988 2750 50  0001 C CNN
@@
 AR Path="/5F387075/60ECB2D9" Ref="#PWR?"  Part="1"
 AR Path="/60E4937F/60ECB2D9" Ref="#PWR?"  Part="1"
-AR Path="/60EC8491/60ECB2D9" Ref="#PWR0110"  Part="1"
-F 0 "#PWR0110" H 4950 2850 50  0001 C CNN
+AR Path="/60EC8491/60ECB2D9" Ref="#PWR0121"  Part="1"
+F 0 "#PWR0121" H 4950 2850 50  0001 C CNN
 F 1 "GND" H 4955 2927 50  0000 C CNN
 F 2 "" H 4950 3100 50  0001 C CNN
@@
 AR Path="/5F387075/60ECB715" Ref="#PWR?"  Part="1"
 AR Path="/60E4937F/60ECB715" Ref="#PWR?"  Part="1"
-AR Path="/60EC8491/60ECB715" Ref="#PWR0111"  Part="1"
-F 0 "#PWR0111" H 5300 3850 50  0001 C CNN
+AR Path="/60EC8491/60ECB715" Ref="#PWR0122"  Part="1"
+F 0 "#PWR0122" H 5300 3850 50  0001 C CNN
 F 1 "GND" H 5305 3927 50  0000 C CNN
 F 2 "" H 5300 4100 50  0001 C CNN
@@
 AR Path="/5F387075/60ED7D95" Ref="R?"  Part="1"
 AR Path="/60E4937F/60ED7D95" Ref="R?"  Part="1"
-AR Path="/60EC8491/60ED7D95" Ref="R69"  Part="1"
-F 0 "R69" H 6270 3696 50  0000 L CNN
+AR Path="/60EC8491/60ED7D95" Ref="R67"  Part="1"
+F 0 "R67" H 6270 3696 50  0000 L CNN
 F 1 "120" H 6270 3605 50  0000 L CNN
 F 2 "Resistor_SMD:R_0201_0603Metric" V 6130 3650 50  0001 C CNN
@@
 	5850 3500 6200 3500
 $Comp
-L Connector_Generic:Conn_01x02 J5
+L Connector_Generic:Conn_01x02 J10
 U 1 1 60EDAE2F
 P 6800 3600
-F 0 "J5" H 6880 3592 50  0000 L CNN
+F 0 "J10" H 6880 3592 50  0000 L CNN
 F 1 "Conn_01x02" H 6880 3501 50  0000 L CNN
-F 2 "" H 6800 3600 50  0001 C CNN
+F 2 "Connector_Hirose:Hirose_DF13-02P-1.25DSA_1x02_P1.25mm_Vertical" H 6800 3600 50  0001 C CNN
 F 3 "~" H 6800 3600 50  0001 C CNN
 	1    6800 3600

Commit message: First complete release. No EtherCAT, IO ready to be connected.
Parts:
- renumbered C141 to C91, J10 to J9, R67 to R37, U10 to U9
Changed lines of the file:
@@
 $Descr A4 11693 8268
 encoding utf-8
-Sheet 6 10
+Sheet 5 10
 Title "Open MOtor DRiver Initiative (OMODRI)"
 Date ""
@@
 $EndDescr
 $Comp
-L Interface_CAN_LIN:TCAN332G U10
+L Interface_CAN_LIN:TCAN332G U?
 U 1 1 60EC8ED3
 P 5300 3650
-F 0 "U10" H 5400 4100 50  0000 C CNN
+AR Path="/60EC8491/60EC8ED3" Ref="U?"  Part="1"
+AR Path="/5F5B575B/60EC8ED3" Ref="U9"  Part="1"
+F 0 "U9" H 5400 4100 50  0000 C CNN
 F 1 "TCAN332G" H 5550 4000 50  0000 C CNN
 F 2 "Package_TO_SOT_SMD:TSOT-23-8" H 5300 3150 50  0001 C CIN
@@
 AR Path="/5F387075/60ECB2D3" Ref="C?"  Part="1"
 AR Path="/60E4937F/60ECB2D3" Ref="C?"  Part="1"
-AR Path="/60EC8491/60ECB2D3" Ref="C141"  Part="1"
-F 0 "C141" H 5050 3000 50  0000 L CNN
+AR Path="/60EC8491/60ECB2D3" Ref="C?"  Part="1"
+AR Path="/5F5B575B/60ECB2D3" Ref="C91"  Part="1"
+F 0 "C91" H 5050 3000 50  0000 L CNN
 F 1 "100nF" H 5050 2900 50  0000 L CNN
 F 2 "Capacitor_SMD:C_0201_0603Metric" H 4988 2750 50  0001 C CNN
@@
 AR Path="/5F387075/60ECB2D9" Ref="#PWR?"  Part="1"
 AR Path="/60E4937F/60ECB2D9" Ref="#PWR?"  Part="1"
-AR Path="/60EC8491/60ECB2D9" Ref="#PWR0121"  Part="1"
-F 0 "#PWR0121" H 4950 2850 50  0001 C CNN
+AR Path="/60EC8491/60ECB2D9" Ref="#PWR?"  Part="1"
+AR Path="/5F5B575B/60ECB2D9" Ref="#PWR092"  Part="1"
+F 0 "#PWR092" H 4950 2850 50  0001 C CNN
 F 1 "GND" H 4955 2927 50  0000 C CNN
 F 2 "" H 4950 3100 50  0001 C CNN
@@
 AR Path="/5F387075/60ECB715" Ref="#PWR?"  Part="1"
 AR Path="/60E4937F/60ECB715" Ref="#PWR?"  Part="1"
-AR Path="/60EC8491/60ECB715" Ref="#PWR0122"  Part="1"
-F 0 "#PWR0122" H 5300 3850 50  0001 C CNN
+AR Path="/60EC8491/60ECB715" Ref="#PWR?"  Part="1"
+AR Path="/5F5B575B/60ECB715" Ref="#PWR093"  Part="1"
+F 0 "#PWR093" H 5300 3850 50  0001 C CNN
 F 1 "GND" H 5305 3927 50  0000 C CNN
 F 2 "" H 5300 4100 50  0001 C CNN
@@
 AR Path="/5F387075/60ED7D95" Ref="R?"  Part="1"
 AR Path="/60E4937F/60ED7D95" Ref="R?"  Part="1"
-AR Path="/60EC8491/60ED7D95" Ref="R67"  Part="1"
-F 0 "R67" H 6270 3696 50  0000 L CNN
+AR Path="/60EC8491/60ED7D95" Ref="R?"  Part="1"
+AR Path="/5F5B575B/60ED7D95" Ref="R37"  Part="1"
+F 0 "R37" H 6270 3696 50  0000 L CNN
 F 1 "120" H 6270 3605 50  0000 L CNN
 F 2 "Resistor_SMD:R_0201_0603Metric" V 6130 3650 50  0001 C CNN
@@
 	5850 3500 6200 3500
 $Comp
-L Connector_Generic:Conn_01x02 J10
+L Connector_Generic:Conn_01x02 J?
 U 1 1 60EDAE2F
 P 6800 3600
-F 0 "J10" H 6880 3592 50  0000 L CNN
+AR Path="/60EC8491/60EDAE2F" Ref="J?"  Part="1"
+AR Path="/5F5B575B/60EDAE2F" Ref="J9"  Part="1"
+F 0 "J9" H 6880 3592 50  0000 L CNN
 F 1 "Conn_01x02" H 6880 3501 50  0000 L CNN
 F 2 "Connector_Hirose:Hirose_DF13-02P-1.25DSA_1x02_P1.25mm_Vertical" H 6800 3600 50  0001 C CNN

Commit message: Update of the schematics. Driver and power files split. Placement starting.
Parts:
- J7: renamed from J9; DigiKey (none) -> DF13-2P-1.25DSA(75)-ND; Farnell (none) -> 2427585; Mouser (none) -> 798-DF13-2P-125DSA75; Part No (none) -> DF13-2P-1.25DSA(75); RS (none) -> 188-6248
- renumbered C91 to C67, R37 to R21, U9 to U8
Changed lines of the file:
@@
 $Descr A4 11693 8268
 encoding utf-8
-Sheet 5 10
+Sheet 5 17
 Title "Open MOtor DRiver Initiative (OMODRI)"
 Date ""
@@
 P 5300 3650
 AR Path="/60EC8491/60EC8ED3" Ref="U?"  Part="1"
-AR Path="/5F5B575B/60EC8ED3" Ref="U9"  Part="1"
-F 0 "U9" H 5400 4100 50  0000 C CNN
+AR Path="/5F5B575B/60EC8ED3" Ref="U8"  Part="1"
+F 0 "U8" H 5400 4100 50  0000 C CNN
 F 1 "TCAN332G" H 5550 4000 50  0000 C CNN
 F 2 "Package_TO_SOT_SMD:TSOT-23-8" H 5300 3150 50  0001 C CIN
@@
 AR Path="/60E4937F/60ECB2D3" Ref="C?"  Part="1"
 AR Path="/60EC8491/60ECB2D3" Ref="C?"  Part="1"
-AR Path="/5F5B575B/60ECB2D3" Ref="C91"  Part="1"
-F 0 "C91" H 5050 3000 50  0000 L CNN
+AR Path="/5F5B575B/60ECB2D3" Ref="C67"  Part="1"
+F 0 "C67" H 5050 3000 50  0000 L CNN
 F 1 "100nF" H 5050 2900 50  0000 L CNN
 F 2 "Capacitor_SMD:C_0201_0603Metric" H 4988 2750 50  0001 C CNN
@@
 AR Path="/60E4937F/60ECB2D9" Ref="#PWR?"  Part="1"
 AR Path="/60EC8491/60ECB2D9" Ref="#PWR?"  Part="1"
-AR Path="/5F5B575B/60ECB2D9" Ref="#PWR092"  Part="1"
-F 0 "#PWR092" H 4950 2850 50  0001 C CNN
+AR Path="/5F5B575B/60ECB2D9" Ref="#PWR067"  Part="1"
+F 0 "#PWR067" H 4950 2850 50  0001 C CNN
 F 1 "GND" H 4955 2927 50  0000 C CNN
 F 2 "" H 4950 3100 50  0001 C CNN
@@
 AR Path="/60E4937F/60ECB715" Ref="#PWR?"  Part="1"
 AR Path="/60EC8491/60ECB715" Ref="#PWR?"  Part="1"
-AR Path="/5F5B575B/60ECB715" Ref="#PWR093"  Part="1"
-F 0 "#PWR093" H 5300 3850 50  0001 C CNN
+AR Path="/5F5B575B/60ECB715" Ref="#PWR068"  Part="1"
+F 0 "#PWR068" H 5300 3850 50  0001 C CNN
 F 1 "GND" H 5305 3927 50  0000 C CNN
 F 2 "" H 5300 4100 50  0001 C CNN
@@
 AR Path="/60E4937F/60ED7D95" Ref="R?"  Part="1"
 AR Path="/60EC8491/60ED7D95" Ref="R?"  Part="1"
-AR Path="/5F5B575B/60ED7D95" Ref="R37"  Part="1"
-F 0 "R37" H 6270 3696 50  0000 L CNN
+AR Path="/5F5B575B/60ED7D95" Ref="R21"  Part="1"
+F 0 "R21" H 6270 3696 50  0000 L CNN
 F 1 "120" H 6270 3605 50  0000 L CNN
 F 2 "Resistor_SMD:R_0201_0603Metric" V 6130 3650 50  0001 C CNN
@@
 P 6800 3600
 AR Path="/60EC8491/60EDAE2F" Ref="J?"  Part="1"
-AR Path="/5F5B575B/60EDAE2F" Ref="J9"  Part="1"
-F 0 "J9" H 6880 3592 50  0000 L CNN
+AR Path="/5F5B575B/60EDAE2F" Ref="J7"  Part="1"
+F 0 "J7" H 6880 3592 50  0000 L CNN
 F 1 "Conn_01x02" H 6880 3501 50  0000 L CNN
 F 2 "Connector_Hirose:Hirose_DF13-02P-1.25DSA_1x02_P1.25mm_Vertical" H 6800 3600 50  0001 C CNN
-F 3 "~" H 6800 3600 50  0001 C CNN
+F 3 "https://www.hirose.com/product/document?clcode=&productname=&series=DF13&documenttype=Catalog&lang=en&documentid=D31687_en" H 6800 3600 50  0001 C CNN
+F 4 "DF13-2P-1.25DSA(75)-ND" H 6800 3600 50  0001 C CNN "DigiKey"
+F 5 "2427585" H 6800 3600 50  0001 C CNN "Farnell"
+F 6 "798-DF13-2P-125DSA75" H 6800 3600 50  0001 C CNN "Mouser"
+F 7 "DF13-2P-1.25DSA(75)" H 6800 3600 50  0001 C CNN "Part No"
+F 8 "188-6248" H 6800 3600 50  0001 C CNN "RS"
 	1    6800 3600
 	1    0    0    -1

Commit message: First release of the fully routed OMODRI PCB from LAAS. (8 layers)
Parts:
- J7: footprint Connector_Hirose:Hirose_DF13-02P-1.25DSA_1x02_P1.25mm_Vertical -> udriver3:Hirose_DF13-02P-1.25DSA_1x02_P1.25mm_Vertical
Changed lines of the file:
@@
 $Descr A4 11693 8268
 encoding utf-8
-Sheet 8 17
+Sheet 8 19
 Title "Open MOtor DRiver Initiative (OMODRI)"
 Date ""
@@
 F 0 "J7" H 6880 3592 50  0000 L CNN
 F 1 "Conn_01x02" H 6880 3501 50  0000 L CNN
-F 2 "Connector_Hirose:Hirose_DF13-02P-1.25DSA_1x02_P1.25mm_Vertical" H 6800 3600 50  0001 C CNN
+F 2 "udriver3:Hirose_DF13-02P-1.25DSA_1x02_P1.25mm_Vertical" H 6800 3600 50  0001 C CNN
 F 3 "https://www.hirose.com/product/document?clcode=&productname=&series=DF13&documenttype=Catalog&lang=en&documentid=D31687_en" H 6800 3600 50  0001 C CNN
 F 4 "DF13-2P-1.25DSA(75)-ND" H 6800 3600 50  0001 C CNN "DigiKey"
