File: hardware/udriver3/OMODRI_power.sch (KiCad schematic (older format))
At the start: 64 parts, among them U3 LMR36015

Commit message: Update of the BOM. Not yet finished.
Parts:
- added C87, C95: 22uF, Capacitor_SMD:C_0603_1608Metric, symbol Device:C
- added C89: 100nF, Capacitor_SMD:C_0201_0603Metric, symbol Device:C
- added C94: 1uF, Capacitor_SMD:C_0201_0603Metric, symbol Device:C
- added C97: 22uF, symbol Device:C
- added FB1, FB2, FB3: Ferrite_Bead_Small, symbol Device:Ferrite_Bead_Small
- added U7: REF6230, symbol omodri_lib:REF6230
- C45, C46, C47, C48, C49, C50, C51, C52, C53, C54, C55, C56, C58, C59, C60, C61, C64, C65, C66, C67, C70, C73, C76, C79: renamed from C?; footprint (none) -> Capacitor_SMD:C_0201_0603Metric; DigiKey (none) -> 490-14450-1-ND; Farnell (none) -> 2990681; Mouser (none) -> 81-GRM033C71A104KE4D; Part No (none) -> GRM033C71A104KE14D; RS (none) -> 185-1751; Rated Voltage (none) -> 10V
- C62, C68, C69, C71, C72, C74, C75: renamed from C?; footprint (none) -> Capacitor_SMD:C_0201_0603Metric; DigiKey (none) -> 490-13219-1-ND; Farnell (none) -> 3238032; Mouser (none) -> 81-GRM033C81A105ME5D; Part No (none) -> GRM033C81A105ME05D; Rated Voltage (none) -> 10V
- C77, C78, C80, C81: renamed from C?; footprint (none) -> Capacitor_SMD:C_0402_1005Metric; DigiKey (none) -> 490-13811-1-ND; Farnell (none) -> 2218854; Mouser (none) -> 81-GRM155R60J106ME4D; Part No (none) -> GRM155R60J106ME44D; RS (none) -> 846-7274; Rated Voltage (none) -> 6.3V
- C82: renamed from C45; value 4.7uF -> 10uF; Rated Voltage (none) -> 100V
- C83: renamed from C46; value 220nF -> 100nF; Rated Voltage (none) -> 100V
- C84: renamed from C47; value 220nF -> 100nF; Rated Voltage (none) -> 100V
- C85, C86, C91, C92: renamed from C?; value 15uF -> 22uF; footprint (none) -> Capacitor_SMD:C_0603_1608Metric; DigiKey (none) -> 490-10476-1-ND; Farnell (none) -> 2426957; Mouser (none) -> 81-GRM188R61A226ME5D; Part No (none) -> GRM188R61A226ME15D; RS (none) -> 884-7258; Rated Voltage (none) -> 10V
- C96: renamed from C51; value 15uF -> 22uF; footprint (none) -> Capacitor_SMD:C_0603_1608Metric; DigiKey (none) -> 490-10476-1-ND; Farnell (none) -> 2426957; Mouser (none) -> 81-GRM188R61A226ME5D; Part No (none) -> GRM188R61A226ME15D; RS (none) -> 884-7258; Rated Voltage (none) -> 10V
- C98: renamed from C52; value 15uF -> 22uF; footprint (none) -> Capacitor_SMD:C_0603_1608Metric; DigiKey (none) -> 490-10476-1-ND; Farnell (none) -> 2426957; Mouser (none) -> 81-GRM188R61A226ME5D; Part No (none) -> GRM188R61A226ME15D; RS (none) -> 884-7258; Rated Voltage (none) -> 10V
- C99: renamed from C53; value 15uF -> 22uF; footprint (none) -> Capacitor_SMD:C_0603_1608Metric; DigiKey (none) -> 490-10476-1-ND; Farnell (none) -> 2426957; Mouser (none) -> 81-GRM188R61A226ME5D; Part No (none) -> GRM188R61A226ME15D; RS (none) -> 884-7258; Rated Voltage (none) -> 10V
- L3: renamed from L1; value 10uH -> 6.8uH
- U3: renamed from U?; footprint BGA_DZWTS_TEX -> udriver3:F28388DZWTS
- U5: renamed from U?; footprint (none) -> udriver3:TPS62088YFPR; DigiKey (none) -> 296-52015-2-ND; Mouser (none) -> 595-TPS6208833YFPT; Part No (none) -> TPS6208833YFPT
- U6: renamed from U?; footprint (none) -> udriver3:TPS62088YFPR; DigiKey (none) -> 296-52014-2-ND; Mouser (none) -> 595-TPS6208812YFPT; Part No (none) -> TPS6208812YFPT
- gave numbers to parts that had none: 7
- renumbered C48 to C88, C49 to C90, C50 to C93, R29 to R32, R30 to R33, R31 to R34, U3 to U4
Connections:
- net labels added: REF_3V0
- wire segments 487 -> 524
Other:
- moved on the sheet: C57, C58, C59, C63, C64, C65, C91, C92, U3B

Commit message: Power supply distribution updated.
Parts:
- removed C50, C52, C60: 100nF, Capacitor_SMD:C_0201_0603Metric, symbol Device:C
- removed C97: 22uF, symbol Device:C
- removed C98, C99: 22uF, Capacitor_SMD:C_0603_1608Metric, symbol Device:C
- removed L1, L2: 330nH, symbol Device:L
- removed L3: 6.8uH, symbol Device:L
- removed U4: LMR36015, symbol omodri_lib:LMR36015
- removed U5: TPS6208833, udriver3:TPS62088YFPR, symbol omodri_lib:TPS6208833
- removed U6: TPS6208812, udriver3:TPS62088YFPR, symbol omodri_lib:TPS6208812
- added C45: 10uF, Capacitor_SMD:C_1210_3225Metric, symbol Device:C
- added C89, C94: 10uF, Capacitor_SMD:C_0603_1608Metric, symbol Device:C
- added R29: 150k, Resistor_SMD:R_0201_0603Metric, symbol Device:R
- added R35: 100k, Resistor_SMD:R_0201_0603Metric, symbol Device:R
- added R36: 5.11k, Resistor_SMD:R_0201_0603Metric, symbol Device:R
- added U3, U4: TPSM82821, symbol omodri_lib:TPSM82821
- added U6: LMZ36002, udriver3:LMZ36002RVQR, symbol omodri_lib:LMZ36002
- C46, C47, C48, C53, C56, C58: value 100nF -> 10uF; footprint Capacitor_SMD:C_0201_0603Metric -> Capacitor_SMD:C_0603_1608Metric; DigiKey 490-14450-1-ND -> 490-10475-1-ND; Farnell 2990681 -> 2456110; Mouser 81-GRM033C71A104KE4D -> 81-GRM188R61A106ME9D; Part No GRM033C71A104KE14D -> GRM188R61A106ME69D; RS 185-1751 -> 113-8702
- C49: footprint Capacitor_SMD:C_0201_0603Metric -> Capacitor_SMD:C_0805_2012Metric; DigiKey 490-14450-1-ND -> 490-3285-1-ND; Farnell 2990681 -> 1828921; Mouser 81-GRM033C71A104KE4D -> 81-GRM188R72A104KA35; Part No GRM033C71A104KE14D -> GRM188R72A104KA35D; RS 185-1751 -> (none); Rated Voltage 10V -> 100V
- C51: value 100nF -> 47nF; footprint Capacitor_SMD:C_0201_0603Metric -> Capacitor_SMD:C_0603_1608Metric; DigiKey 490-14450-1-ND -> 445-6032-1-ND; Farnell 2990681 -> 2906791; Mouser 81-GRM033C71A104KE4D -> 810-C1608X7S2A473K; Part No GRM033C71A104KE14D -> C1608X7S2A473K080AB; RS 185-1751 -> (none); Rated Voltage 10V -> 100V
- C54: value 100nF -> 560pF; DigiKey 490-14450-1-ND -> 490-14862-1-ND; Farnell 2990681 -> (none); Mouser 81-GRM033C71A104KE4D -> 81-GRM0335C1E561JA1D; Part No GRM033C71A104KE14D -> GRM0335C1E561JA01D; RS 185-1751 -> (none); Rated Voltage 10V -> 25V
- C55: value 100nF -> 120pF; DigiKey 490-14450-1-ND -> 490-7221-1-ND; Farnell 2990681 -> 2990619; Mouser 81-GRM033C71A104KE4D -> 81-GRM0335C1H121JA1D; Part No GRM033C71A104KE14D -> GRM0335C1H121JA01D; RS 185-1751 -> 185-2011; Rated Voltage 10V -> 50V
- C57: value 2.2uF -> 10uF; footprint (none) -> Capacitor_SMD:C_0603_1608Metric; DigiKey (none) -> 490-10475-1-ND; Farnell (none) -> 2456110; Mouser (none) -> 81-GRM188R61A106ME9D; Part No (none) -> GRM188R61A106ME69D; RS (none) -> 113-8702; Rated Voltage (none) -> 10V
- C59: value 100nF -> 100uF; footprint Capacitor_SMD:C_0201_0603Metric -> Capacitor_SMD:C_1206_3216Metric; DigiKey 490-14450-1-ND -> 445-6007-2-ND; Farnell 2990681 -> 2211193; Mouser 81-GRM033C71A104KE4D -> 810-C3216X5R1A107M; Part No GRM033C71A104KE14D -> C3216X5R1A107M160AC; RS 185-1751 -> 788-3057
- C62, C68, C69, C74, C75: value 1uF -> 100nF; DigiKey 490-13219-1-ND -> 490-14450-1-ND; Farnell 3238032 -> 2990681; Mouser 81-GRM033C81A105ME5D -> 81-GRM033C71A104KE4D; Part No GRM033C81A105ME05D -> GRM033C71A104KE14D; RS (none) -> 185-1751
- C63: value 2.2uF -> 100nF; footprint (none) -> Capacitor_SMD:C_0201_0603Metric; DigiKey (none) -> 490-14450-1-ND; Farnell (none) -> 2990681; Mouser (none) -> 81-GRM033C71A104KE4D; Part No (none) -> GRM033C71A104KE14D; RS (none) -> 185-1751; Rated Voltage (none) -> 10V
- C71: value 1uF -> 10uF; footprint Capacitor_SMD:C_0201_0603Metric -> Capacitor_SMD:C_0603_1608Metric; DigiKey 490-13219-1-ND -> 490-10475-1-ND; Farnell 3238032 -> 2456110; Mouser 81-GRM033C81A105ME5D -> 81-GRM188R61A106ME9D; Part No GRM033C81A105ME05D -> GRM188R61A106ME69D; RS (none) -> 113-8702
- C73: value 100nF -> 1uF; DigiKey 490-14450-1-ND -> 490-13219-1-ND; Farnell 2990681 -> 3238032; Mouser 81-GRM033C71A104KE4D -> 81-GRM033C81A105ME5D; Part No GRM033C71A104KE14D -> GRM033C81A105ME05D; RS 185-1751 -> (none)
- C77, C78, C81: value 10uF -> 100nF; footprint Capacitor_SMD:C_0402_1005Metric -> Capacitor_SMD:C_0201_0603Metric; DigiKey 490-13811-1-ND -> 490-14450-1-ND; Farnell 2218854 -> 2990681; Mouser 81-GRM155R60J106ME4D -> 81-GRM033C71A104KE4D; Part No GRM155R60J106ME44D -> GRM033C71A104KE14D; RS 846-7274 -> 185-1751; Rated Voltage 6.3V -> 10V
- C80: value 10uF -> 1uF; footprint Capacitor_SMD:C_0402_1005Metric -> Capacitor_SMD:C_0201_0603Metric; DigiKey 490-13811-1-ND -> 490-13219-1-ND; Farnell 2218854 -> 3238032; Mouser 81-GRM155R60J106ME4D -> 81-GRM033C81A105ME5D; Part No GRM155R60J106ME44D -> GRM033C81A105ME05D; RS 846-7274 -> (none); Rated Voltage 6.3V -> 10V
- C82: value 10uF -> 1uF; footprint (none) -> Capacitor_SMD:C_0201_0603Metric; DigiKey (none) -> 490-13219-1-ND; Farnell (none) -> 3238032; Mouser (none) -> 81-GRM033C81A105ME5D; Part No (none) -> GRM033C81A105ME05D; Rated Voltage 100V -> 10V
- C83: value 100nF -> 1uF; footprint (none) -> Capacitor_SMD:C_0201_0603Metric; DigiKey (none) -> 490-13219-1-ND; Farnell (none) -> 3238032; Mouser (none) -> 81-GRM033C81A105ME5D; Part No (none) -> GRM033C81A105ME05D; Rated Voltage 100V -> 10V
- C84: footprint (none) -> Capacitor_SMD:C_0201_0603Metric; DigiKey (none) -> 490-14450-1-ND; Farnell (none) -> 2990681; Mouser (none) -> 81-GRM033C71A104KE4D; Part No (none) -> GRM033C71A104KE14D; RS (none) -> 185-1751; Rated Voltage 100V -> 10V
- C85, C86, C91: value 22uF -> 1uF; footprint Capacitor_SMD:C_0603_1608Metric -> Capacitor_SMD:C_0201_0603Metric; DigiKey 490-10476-1-ND -> 490-13219-1-ND; Farnell 2426957 -> 3238032; Mouser 81-GRM188R61A226ME5D -> 81-GRM033C81A105ME5D; Part No GRM188R61A226ME15D -> GRM033C81A105ME05D; RS 884-7258 -> (none)
- C87, C95: value 22uF -> 100nF; footprint Capacitor_SMD:C_0603_1608Metric -> Capacitor_SMD:C_0201_0603Metric; DigiKey 490-10476-1-ND -> 490-14450-1-ND; Farnell 2426957 -> 2990681; Mouser 81-GRM188R61A226ME5D -> 81-GRM033C71A104KE4D; Part No GRM188R61A226ME15D -> GRM033C71A104KE14D; RS 884-7258 -> 185-1751
- C88: footprint (none) -> Capacitor_SMD:C_0201_0603Metric; DigiKey (none) -> 490-13219-1-ND; Farnell (none) -> 3238032; Mouser (none) -> 81-GRM033C81A105ME5D; Part No (none) -> GRM033C81A105ME05D; Rated Voltage (none) -> 10V
- C90: footprint (none) -> Capacitor_SMD:C_0201_0603Metric; DigiKey (none) -> 490-14450-1-ND; Farnell (none) -> 2990681; Mouser (none) -> 81-GRM033C71A104KE4D; Part No (none) -> GRM033C71A104KE14D; RS (none) -> 185-1751; Rated Voltage (none) -> 10V
- C92, C96: value 22uF -> 10uF; DigiKey 490-10476-1-ND -> 490-10475-1-ND; Farnell 2426957 -> 2456110; Mouser 81-GRM188R61A226ME5D -> 81-GRM188R61A106ME9D; Part No GRM188R61A226ME15D -> GRM188R61A106ME69D; RS 884-7258 -> 113-8702
- C93: value 20pF -> 100nF; footprint (none) -> Capacitor_SMD:C_0201_0603Metric; DigiKey (none) -> 490-14450-1-ND; Farnell (none) -> 2990681; Mouser (none) -> 81-GRM033C71A104KE4D; Part No (none) -> GRM033C71A104KE14D; RS (none) -> 185-1751; Rated Voltage (none) -> 10V
- R30, R31, R32: footprint (none) -> Resistor_SMD:R_0201_0603Metric; DigiKey (none) -> P122655CT-ND; Farnell (none) -> 2302389; Mouser (none) -> 667-ERJ-1GNF1003C; Part No (none) -> ERJ-1GNF1003C; RS (none) -> 179-7130
- R33: value 100k -> 22k; footprint (none) -> Resistor_SMD:R_0201_0603Metric; DigiKey (none) -> P122833CT-ND; Farnell (none) -> 2302371; Mouser (none) -> 667-ERJ-1GNF2202C; Part No (none) -> ERJ-1GNF2202C; RS (none) -> 179-7156
- R34: value 24.9k -> 100k; footprint (none) -> Resistor_SMD:R_0201_0603Metric; DigiKey (none) -> P122655CT-ND; Farnell (none) -> 2302389; Mouser (none) -> 667-ERJ-1GNF1003C; Part No (none) -> ERJ-1GNF1003C; RS (none) -> 179-7130
- R37: renamed from R29; footprint (none) -> Resistor_SMD:R_0201_0603Metric; DigiKey (none) -> P123082CT-ND; Farnell (none) -> 2396848; Mouser (none) -> 667-ERJ-1GNF56R0C; Part No (none) -> ERJ-1GNF56R0C
- renumbered C89 to C50, C94 to C52, C45 to C60, U7 to U5, U3 to U7
Connections:
- net labels added: FB_1V2, FB_3V3, GNDA, PH
- wire segments 524 -> 592
- no-connect marks 0 -> 1
Other:
- note added: "CSET=47nF,\nSoft-Start->20ms delay\n"
- note added: "RSET=5.11k\nVout->5.0V"
- note added: "RTSEL=H-Z, RT=150k,\nFreq->269kHz"
- note added: "Vout ≥ 4.5V\nVBSEL->VOUT."
- moved on the sheet: C50, C52, C60, R37, U5, U7A, U7B

Commit message: Updated version with 28388D pin matching PAL design.
Parts:
- removed C46, C47, C56, C57, C58: 10uF, Capacitor_SMD:C_0603_1608Metric, symbol Device:C
- removed C54: 560pF, Capacitor_SMD:C_0201_0603Metric, symbol Device:C
- removed C55: 120pF, Capacitor_SMD:C_0201_0603Metric, symbol Device:C
- removed R30, R31, R32, R34, R35: 100k, Resistor_SMD:R_0201_0603Metric, symbol Device:R
- removed R33: 22k, Resistor_SMD:R_0201_0603Metric, symbol Device:R
- removed U3, U4: TPSM82821, symbol omodri_lib:TPSM82821
- added C106, C107, C80, C81, C82: 10uF, Capacitor_SMD:C_0603_1608Metric, symbol Device:C
- added C116: 100nF, Capacitor_SMD:C_0201_0603Metric, symbol Device:C
- added D3, D4: LED GREEN, LED_SMD:LED_0402_1005Metric, symbol Device:LED
- added R49, R61: 470, Resistor_SMD:R_0201_0603Metric, symbol Device:R
- added R52, R59: 100k, Resistor_SMD:R_0201_0603Metric, symbol Device:R
- added R53: 19.1k, Resistor_SMD:R_0201_0603Metric, symbol Device:R
- added R54, R58: 0, Resistor_SMD:R_0201_0603Metric, symbol Device:R
- added R55, R60: 37.4k, Resistor_SMD:R_0201_0603Metric, symbol Device:R
- added R57: 118k, Resistor_SMD:R_0201_0603Metric, symbol Device:R
- added U5, U6: MAXM17623, udriver3:TPSM82821SILR, symbol omodri_lib:MAXM17623
- added U8: OPA388, Package_TO_SOT_SMD:SOT-23-5, symbol omodri_lib:OPA388
- FB1, FB2, FB3: footprint (none) -> Inductor_SMD:L_0603_1608Metric; DigiKey (none) -> 490-5225-1-ND; Farnell (none) -> 1515753; Mouser (none) -> 81-BLM18SG221TN1D; Part No (none) -> BLM18SG221TN1D; RS (none) -> 792-6271
- R51: renamed from R36; Rated Voltage (none) -> 15
- U3: renamed from U6; footprint udriver3:LMZ36002RVQR -> udrive3:B3QFN_43
- U4: renamed from U7; footprint udriver3:F28388DZWTS -> udrive3:NFBGA_337; DigiKey (none) -> 296-F28388DZWTS-ND; Mouser (none) -> 595-F28388DZWTS; Part No (none) -> F28388DZWTS
- U7: renamed from U5; footprint (none) -> Package_SO:VSSOP-8_3.0x3.0mm_P0.65mm; DigiKey (none) -> 296-44923-1-ND; Farnell (none) -> 2673367; Mouser (none) -> 595-REF6230IDGKT; Part No (none) -> REF6230IDGKT
- renumbered C81 to C100, C84 to C101, C87 to C102, C90 to C103, C93 to C104, C95 to C105, C70 to C108, C76 to C109, C82 to C110, C85 to C111, C88 to C112, C91 to C113, C94 to C114, C96 to C115, C48 to C117, C50 to C118, C52 to C119, C53 to C120, C71 to C70, C77 to C71, C78 to C73, C45 to C74, C49 to C75, C51 to C76, C59 to C77, C73 to C78, C60 to C83, C62 to C84, C64 to C85, C66 to C86, C68 to C87, C74 to C88, C80 to C89, C83 to C90, C86 to C91, C89 to C92, C92 to C93, C61 to C94, C63 to C95, C65 to C96, C67 to C97, C69 to C98, C75 to C99, R29 to R50, R37 to R56
Connections:
- net labels added: FB_5V0, REF_3V0_BUF
- wire segments 592 -> 602
Other:
- moved on the sheet: C100, C101, C102, C103, C104, C105, C108, C109, C110, C111, C112, C113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

Commit message: All footprints are present. DRV with 2 power branches.
Parts:
- removed C106, C107, C80, C81, C82: 10uF, Capacitor_SMD:C_0603_1608Metric, symbol Device:C
- removed D4: LED GREEN, LED_SMD:LED_0402_1005Metric, symbol Device:LED
- removed R52: 100k, Resistor_SMD:R_0201_0603Metric, symbol Device:R
- removed R53: 19.1k, Resistor_SMD:R_0201_0603Metric, symbol Device:R
- removed R57: 118k, Resistor_SMD:R_0201_0603Metric, symbol Device:R
- removed R60: 37.4k, Resistor_SMD:R_0201_0603Metric, symbol Device:R
- removed R61: 470, Resistor_SMD:R_0201_0603Metric, symbol Device:R
- removed U5, U6: MAXM17623, udriver3:TPSM82821SILR, symbol omodri_lib:MAXM17623
- added C115, C116, C117, C89, C90, C91: 10uF, Capacitor_SMD:C_0603_1608Metric, symbol Device:C
- added D5: LED GREEN, LED_SMD:LED_0402_1005Metric, symbol Device:LED
- added R56: 220, Resistor_SMD:R_0201_0603Metric, symbol Device:R
- added U5, U6: MPM3804GG, udrive3:QFN-10_2x2mm_P0.5mm, symbol omodri_lib:MPM3804GG
- R53: renamed from R51; value 5.11k -> 5.1k; footprint Resistor_SMD:R_0201_0603Metric -> Resistor_SMD:R_0402_1005Metric; DigiKey P123055CT-ND -> P5.10KLCT-ND; Farnell 3302998 -> 2302709; Mouser 667-ERJ-1GNF5111C -> 667-ERJ-2RKF5101X; Part No ERJ-1GNF5111C -> ERJ-2RKF5101X; RS (none) -> 732-5536; Rated Voltage 15 -> 50
- R54, R58: value 0 -> 100k; DigiKey P15979CT-ND -> P122655CT-ND; Farnell 2797350 -> 2302389; Mouser 667-ERJ-1GN0R00C -> 667-ERJ-1GNF1003C; Part No ERJ-1GN0R00C -> ERJ-1GNF1003C; RS 176-3574 -> 179-7130
- R55: value 37.4k -> 22.1k; DigiKey P122973CT-ND -> P122837CT-ND; Farnell 3302927 -> 3335196; Mouser 667-ERJ-1GNF3742C -> 667-ERJ-1GNF2212C; Part No ERJ-1GNF3742C -> ERJ-1GNF2212C
- U8: footprint Package_TO_SOT_SMD:SOT-23-5 -> Package_TO_SOT_SMD:TSOT-23-5
- renumbered C91 to C100, C92 to C101, C93 to C102, C94 to C103, C95 to C104, C96 to C105, C97 to C106, C98 to C107, C99 to C108, C100 to C109, C101 to C110, C102 to C111, C103 to C112, C104 to C113, C105 to C114, C108 to C118, C109 to C119, C110 to C120, C111 to C121, C112 to C122, C113 to C123, C114 to C124, C115 to C125, C116 to C126, C117 to C127, C118 to C128, C119 to C129, C120 to C130, C70 to C79, C71 to C80, C72 to C81, C73 to C82, C74 to C83, C75 to C84, C76 to C85, C77 to C86, C78 to C87, C79 to C88, C83 to C92, C84 to C93, C85 to C94, C86 to C95, C87 to C96, C88 to C97, C89 to C98, C90 to C99, D3 to D4, R49 to R51, R50 to R52, R56 to R57
Connections:
- net labels removed: PG_1V2, PG_3V3
- wire segments 602 -> 587
Other:
- moved on the sheet: C100, C101, C102, C103, C104, C105, C106, C107, C108, C109, C110, C111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

Commit message: First complete release. No EtherCAT, IO ready to be connected.
Parts:
- removed C100, C120, C121, C81, C87, C98, C99: 1uF, Capacitor_SMD:C_0201_0603Metric, symbol Device:C
- removed C101, C117, C125, C130, C91: 10uF, Capacitor_SMD:C_0603_1608Metric, symbol Device:C
- removed C83: 10uF, Capacitor_SMD:C_1210_3225Metric, symbol Device:C
- removed C84: 100nF, Capacitor_SMD:C_0805_2012Metric, symbol Device:C
- removed C85: 47nF, Capacitor_SMD:C_0603_1608Metric, symbol Device:C
- removed C86: 100uF, Capacitor_SMD:C_1206_3216Metric, symbol Device:C
- removed C94, C95, C96, C97: 100nF, Capacitor_SMD:C_0201_0603Metric, symbol Device:C
- removed D4: LED GREEN, LED_SMD:LED_0402_1005Metric, symbol Device:LED
- removed R51: 470, Resistor_SMD:R_0201_0603Metric, symbol Device:R
- removed R52: 150k, Resistor_SMD:R_0201_0603Metric, symbol Device:R
- removed R53: 5.1k, Resistor_SMD:R_0402_1005Metric, symbol Device:R
- removed R56: 220, Resistor_SMD:R_0201_0603Metric, symbol Device:R
- removed U3: LMZ36002, udrive3:B3QFN_43, symbol omodri_lib:LMZ36002
- added C27: 10uF, Capacitor_SMD:C_1210_3225Metric, symbol Device:C
- added C28: 100nF, Capacitor_SMD:C_0805_2012Metric, symbol Device:C
- added C29: 10nF, Capacitor_SMD:C_0201_0603Metric, symbol Device:C
- added C30, C43, C76: 1uF, Capacitor_SMD:C_0201_0603Metric, symbol Device:C
- added C31: 22uF, Capacitor_SMD:C_0603_1608Metric, symbol Device:C
- added C32, C34, C38, C48, C49, C50, C51, C52, C66, C67, C80: 100nF, Capacitor_SMD:C_0201_0603Metric, symbol Device:C
- added C42, C75, C77, C78: 10uF, Capacitor_SMD:C_0603_1608Metric, symbol Device:C
- added D3: LED GREEN, LED_SMD:LED_0402_1005Metric, symbol Device:LED
- added L1: 22uH, udrive3:L_coilcraft_LPS62xx, symbol Device:L
- added R19: 100k, Resistor_SMD:R_0201_0603Metric, symbol Device:R
- added R20: 1k, Resistor_SMD:R_0201_0603Metric, symbol Device:R
- added R23: 470, Resistor_SMD:R_0201_0603Metric, symbol Device:R
- added R27, R28, R29: 0.1, Resistor_SMD:R_0201_0603Metric, symbol Device:R
- added TP17, TP18, TP19, TP20, TP21: TestPoint, TestPoint:TestPoint_Pad_D1.0mm, symbol Connector:TestPoint
- added U2: MAX17502FxTB, Package_DFN_QFN:TDFN-10-1EP_2x3mm_P0.5mm_EP0.9x2mm, symbol Regulator_Switching:MAX17501FxTB
- C41: renamed from C90; value 10uF -> 22uF; DigiKey 490-10475-1-ND -> 490-10476-1-ND; Farnell 2456110 -> 2426957; Mouser 81-GRM188R61A106ME9D -> 81-GRM188R61A226ME5D; Part No GRM188R61A106ME69D -> GRM188R61A226ME15D; RS 113-8702 -> 884-7258
- C45: renamed from C116; value 10uF -> 22uF; DigiKey 490-10475-1-ND -> 490-10476-1-ND; Farnell 2456110 -> 2426957; Mouser 81-GRM188R61A106ME9D -> 81-GRM188R61A226ME5D; Part No GRM188R61A106ME69D -> GRM188R61A226ME15D; RS 113-8702 -> 884-7258
- C79: value 10uF -> 100nF; footprint Capacitor_SMD:C_0603_1608Metric -> Capacitor_SMD:C_0201_0603Metric; DigiKey 490-10475-1-ND -> 490-14450-1-ND; Farnell 2456110 -> 2990681; Mouser 81-GRM188R61A106ME9D -> 81-GRM033C71A104KE4D; Part No GRM188R61A106ME69D -> GRM033C71A104KE14D; RS 113-8702 -> 185-1751
- FB1, FB2, FB3: value Ferrite_Bead_Small -> 220R@100MHz
- renumbered C80 to C33, C82 to C35, C124 to C36, C123 to C37, C88 to C39, C89 to C40, C115 to C44, C102 to C46, C122 to C47, C92 to C53, C93 to C54, C103 to C55, C104 to C56, C105 to C57, C106 to C58, C107 to C59, C108 to C60, C109 to C61, C110 to C62, C126 to C63, C118 to C64, C119 to C65, C111 to C68, C112 to C69, C113 to C70, C114 to C71, C127 to C72, C128 to C73, C129 to C74, D5 to D4, R54 to R21, R55 to R22, R58 to R24, R59 to R25, R57 to R26, U4 to U3, U5 to U4, U6 to U5, U7 to U6, U8 to U7
Connections:
- net labels removed: PH
- wire segments 587 -> 528
- no-connect marks 1 -> 0
Other:
- note removed: "CSET=47nF,\nSoft-Start->20ms delay\n"
- note removed: "RSET=5.11k\nVout->5.0V"
- note removed: "RTSEL=H-Z, RT=150k,\nFreq->269kHz"
- note removed: "Vout ≥ 4.5V\nVBSEL->VOUT."
- moved on the sheet: C36, C37, C40, C41, C44, C45, C46, C47, C53, C54, C55, C56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
