File: hardware/udriver3/OMODRI_FSI_RX.sch (KiCad schematic (older format))
At the start: 12 parts, among them J7 Conn_01x08, U14 TPD6E05U06, U15 DSLVDS1048PWR

Commit message: All footprints are present. DRV with 2 power branches.
Parts:
- removed C138: 100nF, Capacitor_SMD:C_0201_0603Metric, symbol Device:C
- removed J7: Conn_01x08, symbol Connector_Generic:Conn_01x08
- removed R81: 10k, Resistor_SMD:R_0201_0603Metric, symbol Device:R
- added J12: Conn_01x07, Connector_Hirose:Hirose_DF13-07P-1.25DSA_1x07_P1.25mm_Vertical, symbol Connector_Generic:Conn_01x07
- R71: renamed from R75; DigiKey (none) -> P122654CT-ND; Farnell (none) -> 2302309; Mouser (none) -> 667-ERJ-1GNF1000C; Part No (none) -> ERJ-1GNF1000C; RS (none) -> 179-7123
- R72: renamed from R76; DigiKey (none) -> P122654CT-ND; Farnell (none) -> 2302309; Mouser (none) -> 667-ERJ-1GNF1000C; Part No (none) -> ERJ-1GNF1000C; RS (none) -> 179-7123
- R73: renamed from R77; DigiKey (none) -> P122654CT-ND; Farnell (none) -> 2302309; Mouser (none) -> 667-ERJ-1GNF1000C; Part No (none) -> ERJ-1GNF1000C; RS (none) -> 179-7123
- U13: renamed from U14; DigiKey (none) -> 296-39349-1-ND; Mouser (none) -> 595-TPD6E05U06RVZR; Part No (none) -> TPD6E05U06RVZR
- U14: renamed from U15; value DSLVDS1048PWR -> DSLVDS1048; DigiKey (none) -> 296-51106-1-ND; Mouser (none) -> 595-DSLVDS1048PWR; Part No (none) -> DSLVDS1048PWR
- renumbered C139 to C146, R78 to R74, R79 to R75, R80 to R76
Connections:
- net labels removed: RX_FSI_EN
- wire segments 72 -> 65
Other:
- moved on the sheet: R74, R75, R76

Commit message: First complete release. No EtherCAT, IO ready to be connected.
Parts:
- renumbered C146 to C92, J12 to J10, R71 to R38, R72 to R39, R73 to R40, R74 to R41, R75 to R42, R76 to R43, U13 to U10, U14 to U11
Changed lines of the file:
@@
 $Descr A4 11693 8268
 encoding utf-8
-Sheet 8 10
+Sheet 6 10
 Title "Open MOtor DRiver Initiative (OMODRI)"
 Date ""
@@
 $EndDescr
 $Comp
-L omodri_lib:DSLVDS1048PWR U14
+L omodri_lib:DSLVDS1048PWR U?
 U 1 1 5F4A731C
 P 4250 3650
-F 0 "U14" H 3700 2800 60  0000 C CNN
+AR Path="/5F497A69/5F4A731C" Ref="U?"  Part="1"
+AR Path="/5F5B5760/5F4A731C" Ref="U11"  Part="1"
+F 0 "U11" H 3700 2800 60  0000 C CNN
 F 1 "DSLVDS1048" H 4050 4600 60  0000 C CNN
 F 2 "Package_SO:TSSOP-16_4.4x5mm_P0.65mm" H 4150 2800 60  0001 C CNN
@@
 $EndComp
 $Comp
-L Device:R R71
+L Device:R R?
 U 1 1 5F4A7322
 P 5350 2900
-F 0 "R71" V 5143 2900 50  0000 C CNN
+AR Path="/5F497A69/5F4A7322" Ref="R?"  Part="1"
+AR Path="/5F5B5760/5F4A7322" Ref="R38"  Part="1"
+F 0 "R38" V 5143 2900 50  0000 C CNN
 F 1 "100" V 5234 2900 50  0000 C CNN
 F 2 "Resistor_SMD:R_0201_0603Metric" V 5280 2900 50  0001 C CNN
@@
 Connection ~ 5100 2850
 $Comp
-L Device:R R72
+L Device:R R?
 U 1 1 5F4A7330
 P 5350 3250
-F 0 "R72" V 5143 3250 50  0000 C CNN
+AR Path="/5F497A69/5F4A7330" Ref="R?"  Part="1"
+AR Path="/5F5B5760/5F4A7330" Ref="R39"  Part="1"
+F 0 "R39" V 5143 3250 50  0000 C CNN
 F 1 "100" V 5234 3250 50  0000 C CNN
 F 2 "Resistor_SMD:R_0201_0603Metric" V 5280 3250 50  0001 C CNN
@@
 Connection ~ 5100 3200
 $Comp
-L Device:R R73
+L Device:R R?
 U 1 1 5F4A733E
 P 5350 3600
-F 0 "R73" V 5143 3600 50  0000 C CNN
+AR Path="/5F497A69/5F4A733E" Ref="R?"  Part="1"
+AR Path="/5F5B5760/5F4A733E" Ref="R40"  Part="1"
+F 0 "R40" V 5143 3600 50  0000 C CNN
 F 1 "100" V 5234 3600 50  0000 C CNN
 F 2 "Resistor_SMD:R_0201_0603Metric" V 5280 3600 50  0001 C CNN
@@
 AR Path="/5F3A3F16/5F4A734D" Ref="#PWR?"  Part="1"
 AR Path="/5F7A5BAE/5F4A734D" Ref="#PWR?"  Part="1"
-AR Path="/5F497A69/5F4A734D" Ref="#PWR0140"  Part="1"
-F 0 "#PWR0140" H 5100 4550 50  0001 C CNN
+AR Path="/5F497A69/5F4A734D" Ref="#PWR?"  Part="1"
+AR Path="/5F5B5760/5F4A734D" Ref="#PWR0100"  Part="1"
+F 0 "#PWR0100" H 5100 4550 50  0001 C CNN
 F 1 "GND" H 5105 4627 50  0000 C CNN
 F 2 "" H 5100 4800 50  0001 C CNN
@@
 AR Path="/5F3A3F16/5F4A7359" Ref="C?"  Part="1"
 AR Path="/5F7A5BAE/5F4A7359" Ref="C?"  Part="1"
-AR Path="/5F497A69/5F4A7359" Ref="C146"  Part="1"
-F 0 "C146" H 5215 4646 50  0000 L CNN
+AR Path="/5F497A69/5F4A7359" Ref="C?"  Part="1"
+AR Path="/5F5B5760/5F4A7359" Ref="C92"  Part="1"
+F 0 "C92" H 5215 4646 50  0000 L CNN
 F 1 "100nF" H 5215 4555 50  0000 L CNN
 F 2 "Capacitor_SMD:C_0201_0603Metric" H 5138 4450 50  0001 C CNN
@@
 AR Path="/5F3A3F16/5F4A73FF" Ref="#PWR?"  Part="1"
 AR Path="/5F7A5BAE/5F4A73FF" Ref="#PWR?"  Part="1"
-AR Path="/5F497A69/5F4A73FF" Ref="#PWR0139"  Part="1"
-F 0 "#PWR0139" H 3250 4550 50  0001 C CNN
+AR Path="/5F497A69/5F4A73FF" Ref="#PWR?"  Part="1"
+AR Path="/5F5B5760/5F4A73FF" Ref="#PWR099"  Part="1"
+F 0 "#PWR099" H 3250 4550 50  0001 C CNN
 F 1 "GND" H 3255 4627 50  0000 C CNN
 F 2 "" H 3250 4800 50  0001 C CNN
@@
 $EndComp
 $Comp
-L Device:R R74
+L Device:R R?
 U 1 1 5F4A740B
 P 2350 4600
-F 0 "R74" H 2280 4554 50  0000 R CNN
+AR Path="/5F497A69/5F4A740B" Ref="R?"  Part="1"
+AR Path="/5F5B5760/5F4A740B" Ref="R41"  Part="1"
+F 0 "R41" H 2280 4554 50  0000 R CNN
 F 1 "10k" H 2280 4645 50  0000 R CNN
 F 2 "Resistor_SMD:R_0201_0603Metric" V 2280 4600 50  0001 C CNN
@@
 $EndComp
 $Comp
-L Device:R R75
+L Device:R R?
 U 1 1 5F4A7416
 P 2650 4600
-F 0 "R75" H 2580 4554 50  0000 R CNN
+AR Path="/5F497A69/5F4A7416" Ref="R?"  Part="1"
+AR Path="/5F5B5760/5F4A7416" Ref="R42"  Part="1"
+F 0 "R42" H 2580 4554 50  0000 R CNN
 F 1 "10k" H 2580 4645 50  0000 R CNN
 F 2 "Resistor_SMD:R_0201_0603Metric" V 2580 4600 50  0001 C CNN
@@
 $EndComp
 $Comp
-L Device:R R76
+L Device:R R?
 U 1 1 5F4A7421
 P 2950 4600
-F 0 "R76" H 2880 4554 50  0000 R CNN
+AR Path="/5F497A69/5F4A7421" Ref="R?"  Part="1"
+AR Path="/5F5B5760/5F4A7421" Ref="R43"  Part="1"
+F 0 "R43" H 2880 4554 50  0000 R CNN
 F 1 "10k" H 2880 4645 50  0000 R CNN
 F 2 "Resistor_SMD:R_0201_0603Metric" V 2880 4600 50  0001 C CNN
@@
 AR Path="/5F3A3F16/5F4A7427" Ref="#PWR?"  Part="1"
 AR Path="/5F7A5BAE/5F4A7427" Ref="#PWR?"  Part="1"
-AR Path="/5F497A69/5F4A7427" Ref="#PWR0136"  Part="1"
-F 0 "#PWR0136" H 2350 4550 50  0001 C CNN
+AR Path="/5F497A69/5F4A7427" Ref="#PWR?"  Part="1"
+AR Path="/5F5B5760/5F4A7427" Ref="#PWR096"  Part="1"
+F 0 "#PWR096" H 2350 4550 50  0001 C CNN
 F 1 "GND" H 2355 4627 50  0000 C CNN
 F 2 "" H 2350 4800 50  0001 C CNN
@@
 AR Path="/5F3A3F16/5F4A742D" Ref="#PWR?"  Part="1"
 AR Path="/5F7A5BAE/5F4A742D" Ref="#PWR?"  Part="1"
-AR Path="/5F497A69/5F4A742D" Ref="#PWR0137"  Part="1"
-F 0 "#PWR0137" H 2650 4550 50  0001 C CNN
+AR Path="/5F497A69/5F4A742D" Ref="#PWR?"  Part="1"
+AR Path="/5F5B5760/5F4A742D" Ref="#PWR097"  Part="1"
+F 0 "#PWR097" H 2650 4550 50  0001 C CNN
 F 1 "GND" H 2655 4627 50  0000 C CNN
 F 2 "" H 2650 4800 50  0001 C CNN
@@
 AR Path="/5F3A3F16/5F4A7433" Ref="#PWR?"  Part="1"
 AR Path="/5F7A5BAE/5F4A7433" Ref="#PWR?"  Part="1"
-AR Path="/5F497A69/5F4A7433" Ref="#PWR0138"  Part="1"
-F 0 "#PWR0138" H 2950 4550 50  0001 C CNN
+AR Path="/5F497A69/5F4A7433" Ref="#PWR?"  Part="1"
+AR Path="/5F5B5760/5F4A7433" Ref="#PWR098"  Part="1"
+F 0 "#PWR098" H 2950 4550 50  0001 C CNN
 F 1 "GND" H 2955 4627 50  0000 C CNN
 F 2 "" H 2950 4800 50  0001 C CNN
@@
 NoConn ~ 5050 4000
 $Comp
-L omodri_lib:TPD6E05U06 U13
+L omodri_lib:TPD6E05U06 U?
 U 1 1 5F4A7484
 P 6850 3250
-F 0 "U13" H 6850 3965 50  0000 C CNN
+AR Path="/5F497A69/5F4A7484" Ref="U?"  Part="1"
+AR Path="/5F5B5760/5F4A7484" Ref="U10"  Part="1"
+F 0 "U10" H 6850 3965 50  0000 C CNN
 F 1 "TPD6E05U06" H 6850 3874 50  0000 C CNN
 F 2 "udrive3:USON_14" V 6850 3250 50  0001 C CNN
@@
 AR Path="/5F3A3F16/5F4A748A" Ref="#PWR?"  Part="1"
 AR Path="/5F7A5BAE/5F4A748A" Ref="#PWR?"  Part="1"
-AR Path="/5F497A69/5F4A748A" Ref="#PWR0135"  Part="1"
-F 0 "#PWR0135" H 6850 4050 50  0001 C CNN
+AR Path="/5F497A69/5F4A748A" Ref="#PWR?"  Part="1"
+AR Path="/5F5B5760/5F4A748A" Ref="#PWR095"  Part="1"
+F 0 "#PWR095" H 6850 4050 50  0001 C CNN
 F 1 "GND" H 6855 4127 50  0000 C CNN
 F 2 "" H 6850 4300 50  0001 C CNN
@@
 AR Path="/5F3A3F16/5F59AE73" Ref="#PWR?"  Part="1"
 AR Path="/5F7A5BAE/5F59AE73" Ref="#PWR?"  Part="1"
-AR Path="/5F497A69/5F59AE73" Ref="#PWR0134"  Part="1"
-F 0 "#PWR0134" H 8500 2650 50  0001 C CNN
+AR Path="/5F497A69/5F59AE73" Ref="#PWR?"  Part="1"
+AR Path="/5F5B5760/5F59AE73" Ref="#PWR094"  Part="1"
+F 0 "#PWR094" H 8500 2650 50  0001 C CNN
 F 1 "GND" V 8500 2700 50  0000 C CNN
 F 2 "" H 8500 2900 50  0001 C CNN
@@
 	2050 2900 2350 2900
 $Comp
-L Connector_Generic:Conn_01x07 J12
+L Connector_Generic:Conn_01x07 J?
 U 1 1 5F6E30FC
 P 8800 3200
-F 0 "J12" H 8750 3600 50  0000 L CNN
+AR Path="/5F497A69/5F6E30FC" Ref="J?"  Part="1"
+AR Path="/5F5B5760/5F6E30FC" Ref="J10"  Part="1"
+F 0 "J10" H 8750 3600 50  0000 L CNN
 F 1 "Conn_01x07" H 8750 2800 50  0000 L CNN
 F 2 "Connector_Hirose:Hirose_DF13-07P-1.25DSA_1x07_P1.25mm_Vertical" H 8800 3200 50  0001 C CNN

Commit message: Update of the schematics. Driver and power files split. Placement starting.
Parts:
- J8: renamed from J10; DigiKey (none) -> DF13-7P-1.25DSA(75)-ND; Mouser (none) -> 798-DF13-7P-125DSA75; Part No (none) -> DF13-7P-1.25DSA(75); RS (none) -> 188-6250
- U9: renamed from U10; footprint udrive3:USON_14 -> udriver3:USON_14
- renumbered C92 to C68, R38 to R22, R39 to R23, R40 to R24, R41 to R25, R42 to R26, R43 to R27, U11 to U10
Changed lines of the file:
@@
 $Descr A4 11693 8268
 encoding utf-8
-Sheet 6 10
+Sheet 6 17
 Title "Open MOtor DRiver Initiative (OMODRI)"
 Date ""
@@
 P 4250 3650
 AR Path="/5F497A69/5F4A731C" Ref="U?"  Part="1"
-AR Path="/5F5B5760/5F4A731C" Ref="U11"  Part="1"
-F 0 "U11" H 3700 2800 60  0000 C CNN
+AR Path="/5F5B5760/5F4A731C" Ref="U10"  Part="1"
+F 0 "U10" H 3700 2800 60  0000 C CNN
 F 1 "DSLVDS1048" H 4050 4600 60  0000 C CNN
 F 2 "Package_SO:TSSOP-16_4.4x5mm_P0.65mm" H 4150 2800 60  0001 C CNN
@@
 P 5350 2900
 AR Path="/5F497A69/5F4A7322" Ref="R?"  Part="1"
-AR Path="/5F5B5760/5F4A7322" Ref="R38"  Part="1"
-F 0 "R38" V 5143 2900 50  0000 C CNN
+AR Path="/5F5B5760/5F4A7322" Ref="R22"  Part="1"
+F 0 "R22" V 5143 2900 50  0000 C CNN
 F 1 "100" V 5234 2900 50  0000 C CNN
 F 2 "Resistor_SMD:R_0201_0603Metric" V 5280 2900 50  0001 C CNN
@@
 P 5350 3250
 AR Path="/5F497A69/5F4A7330" Ref="R?"  Part="1"
-AR Path="/5F5B5760/5F4A7330" Ref="R39"  Part="1"
-F 0 "R39" V 5143 3250 50  0000 C CNN
+AR Path="/5F5B5760/5F4A7330" Ref="R23"  Part="1"
+F 0 "R23" V 5143 3250 50  0000 C CNN
 F 1 "100" V 5234 3250 50  0000 C CNN
 F 2 "Resistor_SMD:R_0201_0603Metric" V 5280 3250 50  0001 C CNN
@@
 P 5350 3600
 AR Path="/5F497A69/5F4A733E" Ref="R?"  Part="1"
-AR Path="/5F5B5760/5F4A733E" Ref="R40"  Part="1"
-F 0 "R40" V 5143 3600 50  0000 C CNN
+AR Path="/5F5B5760/5F4A733E" Ref="R24"  Part="1"
+F 0 "R24" V 5143 3600 50  0000 C CNN
 F 1 "100" V 5234 3600 50  0000 C CNN
 F 2 "Resistor_SMD:R_0201_0603Metric" V 5280 3600 50  0001 C CNN
@@
 AR Path="/5F7A5BAE/5F4A734D" Ref="#PWR?"  Part="1"
 AR Path="/5F497A69/5F4A734D" Ref="#PWR?"  Part="1"
-AR Path="/5F5B5760/5F4A734D" Ref="#PWR0100"  Part="1"
-F 0 "#PWR0100" H 5100 4550 50  0001 C CNN
+AR Path="/5F5B5760/5F4A734D" Ref="#PWR075"  Part="1"
+F 0 "#PWR075" H 5100 4550 50  0001 C CNN
 F 1 "GND" H 5105 4627 50  0000 C CNN
 F 2 "" H 5100 4800 50  0001 C CNN
@@
 AR Path="/5F7A5BAE/5F4A7359" Ref="C?"  Part="1"
 AR Path="/5F497A69/5F4A7359" Ref="C?"  Part="1"
-AR Path="/5F5B5760/5F4A7359" Ref="C92"  Part="1"
-F 0 "C92" H 5215 4646 50  0000 L CNN
+AR Path="/5F5B5760/5F4A7359" Ref="C68"  Part="1"
+F 0 "C68" H 5215 4646 50  0000 L CNN
 F 1 "100nF" H 5215 4555 50  0000 L CNN
 F 2 "Capacitor_SMD:C_0201_0603Metric" H 5138 4450 50  0001 C CNN
@@
 AR Path="/5F7A5BAE/5F4A73FF" Ref="#PWR?"  Part="1"
 AR Path="/5F497A69/5F4A73FF" Ref="#PWR?"  Part="1"
-AR Path="/5F5B5760/5F4A73FF" Ref="#PWR099"  Part="1"
-F 0 "#PWR099" H 3250 4550 50  0001 C CNN
+AR Path="/5F5B5760/5F4A73FF" Ref="#PWR074"  Part="1"
+F 0 "#PWR074" H 3250 4550 50  0001 C CNN
 F 1 "GND" H 3255 4627 50  0000 C CNN
 F 2 "" H 3250 4800 50  0001 C CNN
@@
 P 2350 4600
 AR Path="/5F497A69/5F4A740B" Ref="R?"  Part="1"
-AR Path="/5F5B5760/5F4A740B" Ref="R41"  Part="1"
-F 0 "R41" H 2280 4554 50  0000 R CNN
+AR Path="/5F5B5760/5F4A740B" Ref="R25"  Part="1"
+F 0 "R25" H 2280 4554 50  0000 R CNN
 F 1 "10k" H 2280 4645 50  0000 R CNN
 F 2 "Resistor_SMD:R_0201_0603Metric" V 2280 4600 50  0001 C CNN
@@
 P 2650 4600
 AR Path="/5F497A69/5F4A7416" Ref="R?"  Part="1"
-AR Path="/5F5B5760/5F4A7416" Ref="R42"  Part="1"
-F 0 "R42" H 2580 4554 50  0000 R CNN
+AR Path="/5F5B5760/5F4A7416" Ref="R26"  Part="1"
+F 0 "R26" H 2580 4554 50  0000 R CNN
 F 1 "10k" H 2580 4645 50  0000 R CNN
 F 2 "Resistor_SMD:R_0201_0603Metric" V 2580 4600 50  0001 C CNN
@@
 P 2950 4600
 AR Path="/5F497A69/5F4A7421" Ref="R?"  Part="1"
-AR Path="/5F5B5760/5F4A7421" Ref="R43"  Part="1"
-F 0 "R43" H 2880 4554 50  0000 R CNN
+AR Path="/5F5B5760/5F4A7421" Ref="R27"  Part="1"
+F 0 "R27" H 2880 4554 50  0000 R CNN
 F 1 "10k" H 2880 4645 50  0000 R CNN
 F 2 "Resistor_SMD:R_0201_0603Metric" V 2880 4600 50  0001 C CNN
@@
 AR Path="/5F7A5BAE/5F4A7427" Ref="#PWR?"  Part="1"
 AR Path="/5F497A69/5F4A7427" Ref="#PWR?"  Part="1"
-AR Path="/5F5B5760/5F4A7427" Ref="#PWR096"  Part="1"
-F 0 "#PWR096" H 2350 4550 50  0001 C CNN
+AR Path="/5F5B5760/5F4A7427" Ref="#PWR071"  Part="1"
+F 0 "#PWR071" H 2350 4550 50  0001 C CNN
 F 1 "GND" H 2355 4627 50  0000 C CNN
 F 2 "" H 2350 4800 50  0001 C CNN
@@
 AR Path="/5F7A5BAE/5F4A742D" Ref="#PWR?"  Part="1"
 AR Path="/5F497A69/5F4A742D" Ref="#PWR?"  Part="1"
-AR Path="/5F5B5760/5F4A742D" Ref="#PWR097"  Part="1"
-F 0 "#PWR097" H 2650 4550 50  0001 C CNN
+AR Path="/5F5B5760/5F4A742D" Ref="#PWR072"  Part="1"
+F 0 "#PWR072" H 2650 4550 50  0001 C CNN
 F 1 "GND" H 2655 4627 50  0000 C CNN
 F 2 "" H 2650 4800 50  0001 C CNN
@@
 AR Path="/5F7A5BAE/5F4A7433" Ref="#PWR?"  Part="1"
 AR Path="/5F497A69/5F4A7433" Ref="#PWR?"  Part="1"
-AR Path="/5F5B5760/5F4A7433" Ref="#PWR098"  Part="1"
-F 0 "#PWR098" H 2950 4550 50  0001 C CNN
+AR Path="/5F5B5760/5F4A7433" Ref="#PWR073"  Part="1"
+F 0 "#PWR073" H 2950 4550 50  0001 C CNN
 F 1 "GND" H 2955 4627 50  0000 C CNN
 F 2 "" H 2950 4800 50  0001 C CNN
@@
 P 6850 3250
 AR Path="/5F497A69/5F4A7484" Ref="U?"  Part="1"
-AR Path="/5F5B5760/5F4A7484" Ref="U10"  Part="1"
-F 0 "U10" H 6850 3965 50  0000 C CNN
+AR Path="/5F5B5760/5F4A7484" Ref="U9"  Part="1"
+F 0 "U9" H 6850 3965 50  0000 C CNN
 F 1 "TPD6E05U06" H 6850 3874 50  0000 C CNN
-F 2 "udrive3:USON_14" V 6850 3250 50  0001 C CNN
+F 2 "udriver3:USON_14" V 6850 3250 50  0001 C CNN
 F 3 "https://www.ti.com/lit/ds/symlink/tpd6e05u06.pdf" V 6850 3250 50  0001 C CNN
 F 4 "296-39349-1-ND" H 6850 3250 50  0001 C CNN "DigiKey"
@@
 AR Path="/5F7A5BAE/5F4A748A" Ref="#PWR?"  Part="1"
 AR Path="/5F497A69/5F4A748A" Ref="#PWR?"  Part="1"
-AR Path="/5F5B5760/5F4A748A" Ref="#PWR095"  Part="1"
-F 0 "#PWR095" H 6850 4050 50  0001 C CNN
+AR Path="/5F5B5760/5F4A748A" Ref="#PWR070"  Part="1"
+F 0 "#PWR070" H 6850 4050 50  0001 C CNN
 F 1 "GND" H 6855 4127 50  0000 C CNN
 F 2 "" H 6850 4300 50  0001 C CNN
@@
 AR Path="/5F7A5BAE/5F59AE73" Ref="#PWR?"  Part="1"
 AR Path="/5F497A69/5F59AE73" Ref="#PWR?"  Part="1"
-AR Path="/5F5B5760/5F59AE73" Ref="#PWR094"  Part="1"
-F 0 "#PWR094" H 8500 2650 50  0001 C CNN
+AR Path="/5F5B5760/5F59AE73" Ref="#PWR069"  Part="1"
+F 0 "#PWR069" H 8500 2650 50  0001 C CNN
 F 1 "GND" V 8500 2700 50  0000 C CNN
 F 2 "" H 8500 2900 50  0001 C CNN
@@
 P 8800 3200
 AR Path="/5F497A69/5F6E30FC" Ref="J?"  Part="1"
-AR Path="/5F5B5760/5F6E30FC" Ref="J10"  Part="1"
-F 0 "J10" H 8750 3600 50  0000 L CNN
+AR Path="/5F5B5760/5F6E30FC" Ref="J8"  Part="1"
+F 0 "J8" H 8750 3600 50  0000 L CNN
 F 1 "Conn_01x07" H 8750 2800 50  0000 L CNN
 F 2 "Connector_Hirose:Hirose_DF13-07P-1.25DSA_1x07_P1.25mm_Vertical" H 8800 3200 50  0001 C CNN
-F 3 "~" H 8800 3200 50  0001 C CNN
+F 3 "https://www.hirose.com/product/document?clcode=&productname=&series=DF13&documenttype=Catalog&lang=en&documentid=D31687_en" H 8800 3200 50  0001 C CNN
+F 4 "DF13-7P-1.25DSA(75)-ND" H 8800 3200 50  0001 C CNN "DigiKey"
+F 5 "798-DF13-7P-125DSA75" H 8800 3200 50  0001 C CNN "Mouser"
+F 6 "DF13-7P-1.25DSA(75)" H 8800 3200 50  0001 C CNN "Part No"
+F 7 "188-6250" H 8800 3200 50  0001 C CNN "RS"
 	1    8800 3200
 	1    0    0    -1

Commit message: Update of the schematics. Switches on GPIO72 & GPIO84 are missing. J1, J2 & J14 must be merged and connector placement optimized. TCXO must be changed from 20MHz to 25MHz for EtherCAT compatibility. PCB is partially routed in 6-Layers (mainly power supplies and and transistors). 8-Layers will be necessary.
Connections:
- wire segments 65 -> 69
Other:
- moved on the sheet: J8, R24, U9
