File: hardware/udriver3/OMODRI_FSI_TX.sch (KiCad schematic (older format))
At the start: 7 parts, among them J10 Conn_01x07, U13 TPD6E05U06, U14 DSLVDS1047

Commit message: Update of the µOmodri PCB with Gerber, stencil and assembly files.
Parts:
- J10: DigiKey DF13-7P-1.25DSA(75)-ND -> H2196-ND; Mouser 798-DF13-7P-125DSA75 -> 798-DF13-7P-1.25DSA; Part No DF13-7P-1.25DSA(75) -> DF13-7P-1.25DSA; RS 188-6250 -> (none)
Changed lines of the file:
@@
 F 2 "udriver3:Hirose_DF13-07P-1.25DSA_1x07_P1.25mm_Vertical" H 9525 3175 50  0001 C CNN
 F 3 "https://www.hirose.com/product/document?clcode=&productname=&series=DF13&documenttype=Catalog&lang=en&documentid=D31687_en" H 9525 3175 50  0001 C CNN
-F 4 "DF13-7P-1.25DSA(75)-ND" H 9525 3175 50  0001 C CNN "DigiKey"
-F 5 "798-DF13-7P-125DSA75" H 9525 3175 50  0001 C CNN "Mouser"
-F 6 "DF13-7P-1.25DSA(75)" H 9525 3175 50  0001 C CNN "Part No"
-F 7 "188-6250" H 9525 3175 50  0001 C CNN "RS"
+F 4 "H2196-ND" H 9525 3175 50  0001 C CNN "DigiKey"
+F 5 "798-DF13-7P-1.25DSA" H 9525 3175 50  0001 C CNN "Mouser"
+F 6 "DF13-7P-1.25DSA" H 9525 3175 50  0001 C CNN "Part No"
+F 7 "" H 9525 3175 50  0001 C CNN "RS"
 	1    9525 3175
 	1    0    0    -1
