File: hardware/udriver3/OMODRI_ETHERCAT_CONNECT.sch (KiCad schematic (older format))
At the start: 2 parts, among them J15 ADM6_ADF6, J16 ADM6_ADF6

Commit message: Release 1.1 - Update components values + BOM - Update of J1 pins affectation now matching J2 distribution. - Update gerber files with missing inner layers - Few updates of the PCB layout (J2 redraw + decoupling cap)
Parts:
- J15, J16: footprint footprint:SAMTEC_ADF6-10-03.5-L-4-2-A-TR -> udriver3:ADF6-10-XX.X-XXX-4-X-A-XR
Changed lines of the file:
@@
 F 0 "J16" H 6225 3800 50  0000 L CNN
 F 1 "ADM6_ADF6" H 6225 2700 50  0000 L CNN
-F 2 "footprint:SAMTEC_ADF6-10-03.5-L-4-2-A-TR" H 6225 3250 50  0001 C CNN
+F 2 "udriver3:ADF6-10-XX.X-XXX-4-X-A-XR" H 6225 3250 50  0001 C CNN
 F 3 "http://suddendocs.samtec.com/prints/adf6-xxx-xx.x-xxx-4-x-x-xr-mkt.pdf" H 6225 3250 50  0001 C CNN
 F 4 "612-ADF6-10-03.5-L-4-2-A-TR-ND" H 6225 3250 50  0001 C CNN "DigiKey"
@@
 F 0 "J16" H 7725 3800 50  0000 L CNN
 F 1 "ADM6_ADF6" H 7725 2700 50  0000 L CNN
-F 2 "footprint:SAMTEC_ADF6-10-03.5-L-4-2-A-TR" H 7725 3250 50  0001 C CNN
+F 2 "udriver3:ADF6-10-XX.X-XXX-4-X-A-XR" H 7725 3250 50  0001 C CNN
 F 3 "http://suddendocs.samtec.com/prints/adf6-xxx-xx.x-xxx-4-x-x-xr-mkt.pdf" H 7725 3250 50  0001 C CNN
 F 4 "612-ADF6-10-03.5-L-4-2-A-TR-ND" H 7725 3250 50  0001 C CNN "DigiKey"
@@
 F 0 "J15" H 3150 5300 50  0000 L CNN
 F 1 "ADM6_ADF6" H 3150 4200 50  0000 L CNN
-F 2 "footprint:SAMTEC_ADF6-10-03.5-L-4-2-A-TR" H 3150 4750 50  0001 C CNN
+F 2 "udriver3:ADF6-10-XX.X-XXX-4-X-A-XR" H 3150 4750 50  0001 C CNN
 F 3 "http://suddendocs.samtec.com/prints/adf6-xxx-xx.x-xxx-4-x-x-xr-mkt.pdf" H 3150 4750 50  0001 C CNN
 F 4 "612-ADF6-10-03.5-L-4-2-A-TR-ND" H 3150 4750 50  0001 C CNN "DigiKey"
@@
 F 0 "J15" H 7725 5300 50  0000 L CNN
 F 1 "ADM6_ADF6" H 7725 4200 50  0000 L CNN
-F 2 "footprint:SAMTEC_ADF6-10-03.5-L-4-2-A-TR" H 7725 4750 50  0001 C CNN
+F 2 "udriver3:ADF6-10-XX.X-XXX-4-X-A-XR" H 7725 4750 50  0001 C CNN
 F 3 "http://suddendocs.samtec.com/prints/adf6-xxx-xx.x-xxx-4-x-x-xr-mkt.pdf" H 7725 4750 50  0001 C CNN
 F 4 "612-ADF6-10-03.5-L-4-2-A-TR-ND" H 7725 4750 50  0001 C CNN "DigiKey"
@@
 F 0 "J15" H 6225 5300 50  0000 L CNN
 F 1 "ADM6_ADF6" H 6225 4200 50  0000 L CNN
-F 2 "footprint:SAMTEC_ADF6-10-03.5-L-4-2-A-TR" H 6225 4750 50  0001 C CNN
+F 2 "udriver3:ADF6-10-XX.X-XXX-4-X-A-XR" H 6225 4750 50  0001 C CNN
 F 3 "http://suddendocs.samtec.com/prints/adf6-xxx-xx.x-xxx-4-x-x-xr-mkt.pdf" H 6225 4750 50  0001 C CNN
 F 4 "612-ADF6-10-03.5-L-4-2-A-TR-ND" H 6225 4750 50  0001 C CNN "DigiKey"
@@
 F 0 "J15" H 4650 5300 50  0000 L CNN
 F 1 "ADM6_ADF6" H 4650 4200 50  0000 L CNN
-F 2 "footprint:SAMTEC_ADF6-10-03.5-L-4-2-A-TR" H 4650 4750 50  0001 C CNN
+F 2 "udriver3:ADF6-10-XX.X-XXX-4-X-A-XR" H 4650 4750 50  0001 C CNN
 F 3 "http://suddendocs.samtec.com/prints/adf6-xxx-xx.x-xxx-4-x-x-xr-mkt.pdf" H 4650 4750 50  0001 C CNN
 F 4 "612-ADF6-10-03.5-L-4-2-A-TR-ND" H 4650 4750 50  0001 C CNN "DigiKey"
@@
 F 0 "J16" H 3150 3800 50  0000 L CNN
 F 1 "ADM6_ADF6" H 3150 2700 50  0000 L CNN
-F 2 "footprint:SAMTEC_ADF6-10-03.5-L-4-2-A-TR" H 3150 3250 50  0001 C CNN
+F 2 "udriver3:ADF6-10-XX.X-XXX-4-X-A-XR" H 3150 3250 50  0001 C CNN
 F 3 "http://suddendocs.samtec.com/prints/adf6-xxx-xx.x-xxx-4-x-x-xr-mkt.pdf" H 3150 3250 50  0001 C CNN
 F 4 "612-ADF6-10-03.5-L-4-2-A-TR-ND" H 3150 3250 50  0001 C CNN "DigiKey"
@@
 F 0 "J16" H 4650 3800 50  0000 L CNN
 F 1 "ADM6_ADF6" H 4650 2700 50  0000 L CNN
-F 2 "footprint:SAMTEC_ADF6-10-03.5-L-4-2-A-TR" H 4650 3250 50  0001 C CNN
+F 2 "udriver3:ADF6-10-XX.X-XXX-4-X-A-XR" H 4650 3250 50  0001 C CNN
 F 3 "http://suddendocs.samtec.com/prints/adf6-xxx-xx.x-xxx-4-x-x-xr-mkt.pdf" H 4650 3250 50  0001 C CNN
 F 4 "612-ADF6-10-03.5-L-4-2-A-TR-ND" H 4650 3250 50  0001 C CNN "DigiKey"
