File: hardware/udriver3/OMODRI_ANALOG.sch (KiCad schematic (older format))
At the start: 9 parts, among them U1 TMS320F28388D

Commit message: Released version, with 4mils/4mils for track width and isolation on outer and inner layers 0.45mm for inner and outer annular ring 0.1mm for finished via drill (for Seeed studio increase to 0.2mm) + USB connector added
Parts:
- D10, D12, D13, D2, D6, D7, D8, D9: footprint Diode_SMD:D_0201_0603Metric -> udriver3:D_0201_0603Metric; DigiKey 296-47224-1-ND -> 296-47862-1-ND; Mouser 595-TPD1E04U04DPYR -> 595-TPD1E04U04DPLT; Part No TPD1E04U04DPYT -> TPD1E04U04DPLT
Changed lines of the file:
@@
 $Descr A4 11693 8268
 encoding utf-8
-Sheet 15 19
+Sheet 13 19
 Title ""
 Date ""
@@
 F 0 "D9" H 6100 3450 50  0000 L CNN
 F 1 "TPD1E04U04" H 6100 3375 50  0000 L CNN
-F 2 "Diode_SMD:D_0201_0603Metric" H 6500 3125 50  0001 C CNN
+F 2 "udriver3:D_0201_0603Metric" H 6500 3125 50  0001 C CNN
 F 3 "https://www.ti.com/lit/ds/symlink/tpd1e04u04.pdf" H 6500 3125 50  0001 C CNN
-F 4 "296-47224-1-ND" H 6400 3125 50  0001 C CNN "DigiKey"
-F 5 "595-TPD1E04U04DPYR" H 6400 3125 50  0001 C CNN "Mouser"
-F 6 "TPD1E04U04DPYT" H 6400 3125 50  0001 C CNN "Part No"
+F 4 "296-47862-1-ND" H 6400 3125 50  0001 C CNN "DigiKey"
+F 5 "595-TPD1E04U04DPLT" H 6400 3125 50  0001 C CNN "Mouser"
+F 6 "TPD1E04U04DPLT" H 6400 3125 50  0001 C CNN "Part No"
 	1    6400 3125
 	1    0    0    -1
@@
 F 0 "D10" H 7200 3450 50  0000 L CNN
 F 1 "TPD1E04U04" H 7200 3375 50  0000 L CNN
-F 2 "Diode_SMD:D_0201_0603Metric" H 7600 3125 50  0001 C CNN
+F 2 "udriver3:D_0201_0603Metric" H 7600 3125 50  0001 C CNN
 F 3 "https://www.ti.com/lit/ds/symlink/tpd1e04u04.pdf" H 7600 3125 50  0001 C CNN
-F 4 "296-47224-1-ND" H 7500 3125 50  0001 C CNN "DigiKey"
-F 5 "595-TPD1E04U04DPYR" H 7500 3125 50  0001 C CNN "Mouser"
-F 6 "TPD1E04U04DPYT" H 7500 3125 50  0001 C CNN "Part No"
+F 4 "296-47862-1-ND" H 7500 3125 50  0001 C CNN "DigiKey"
+F 5 "595-TPD1E04U04DPLT" H 7500 3125 50  0001 C CNN "Mouser"
+F 6 "TPD1E04U04DPLT" H 7500 3125 50  0001 C CNN "Part No"
 	1    7500 3125
 	1    0    0    -1
@@
 F 0 "D8" H 8250 3450 50  0000 L CNN
 F 1 "TPD1E04U04" H 8250 3375 50  0000 L CNN
-F 2 "Diode_SMD:D_0201_0603Metric" H 8650 3125 50  0001 C CNN
+F 2 "udriver3:D_0201_0603Metric" H 8650 3125 50  0001 C CNN
 F 3 "https://www.ti.com/lit/ds/symlink/tpd1e04u04.pdf" H 8650 3125 50  0001 C CNN
-F 4 "296-47224-1-ND" H 8550 3125 50  0001 C CNN "DigiKey"
-F 5 "595-TPD1E04U04DPYR" H 8550 3125 50  0001 C CNN "Mouser"
-F 6 "TPD1E04U04DPYT" H 8550 3125 50  0001 C CNN "Part No"
+F 4 "296-47862-1-ND" H 8550 3125 50  0001 C CNN "DigiKey"
+F 5 "595-TPD1E04U04DPLT" H 8550 3125 50  0001 C CNN "Mouser"
+F 6 "TPD1E04U04DPLT" H 8550 3125 50  0001 C CNN "Part No"
 	1    8550 3125
 	1    0    0    -1
@@
 F 0 "D2" H 8225 2475 50  0000 L CNN
 F 1 "TPD1E04U04" H 8225 2400 50  0000 L CNN
-F 2 "Diode_SMD:D_0201_0603Metric" H 8625 2150 50  0001 C CNN
+F 2 "udriver3:D_0201_0603Metric" H 8625 2150 50  0001 C CNN
 F 3 "https://www.ti.com/lit/ds/symlink/tpd1e04u04.pdf" H 8625 2150 50  0001 C CNN
-F 4 "296-47224-1-ND" H 8525 2150 50  0001 C CNN "DigiKey"
-F 5 "595-TPD1E04U04DPYR" H 8525 2150 50  0001 C CNN "Mouser"
-F 6 "TPD1E04U04DPYT" H 8525 2150 50  0001 C CNN "Part No"
+F 4 "296-47862-1-ND" H 8525 2150 50  0001 C CNN "DigiKey"
+F 5 "595-TPD1E04U04DPLT" H 8525 2150 50  0001 C CNN "Mouser"
+F 6 "TPD1E04U04DPLT" H 8525 2150 50  0001 C CNN "Part No"
 	1    8525 2150
 	1    0    0    -1
@@
 F 0 "D7" H 7175 2475 50  0000 L CNN
 F 1 "TPD1E04U04" H 7175 2400 50  0000 L CNN
-F 2 "Diode_SMD:D_0201_0603Metric" H 7575 2150 50  0001 C CNN
+F 2 "udriver3:D_0201_0603Metric" H 7575 2150 50  0001 C CNN
 F 3 "https://www.ti.com/lit/ds/symlink/tpd1e04u04.pdf" H 7575 2150 50  0001 C CNN
-F 4 "296-47224-1-ND" H 7475 2150 50  0001 C CNN "DigiKey"
-F 5 "595-TPD1E04U04DPYR" H 7475 2150 50  0001 C CNN "Mouser"
-F 6 "TPD1E04U04DPYT" H 7475 2150 50  0001 C CNN "Part No"
+F 4 "296-47862-1-ND" H 7475 2150 50  0001 C CNN "DigiKey"
+F 5 "595-TPD1E04U04DPLT" H 7475 2150 50  0001 C CNN "Mouser"
+F 6 "TPD1E04U04DPLT" H 7475 2150 50  0001 C CNN "Part No"
 	1    7475 2150
 	1    0    0    -1
@@
 F 0 "D6" H 6100 2475 50  0000 L CNN
 F 1 "TPD1E04U04" H 6100 2400 50  0000 L CNN
-F 2 "Diode_SMD:D_0201_0603Metric" H 6500 2150 50  0001 C CNN
+F 2 "udriver3:D_0201_0603Metric" H 6500 2150 50  0001 C CNN
 F 3 "https://www.ti.com/lit/ds/symlink/tpd1e04u04.pdf" H 6500 2150 50  0001 C CNN
-F 4 "296-47224-1-ND" H 6400 2150 50  0001 C CNN "DigiKey"
-F 5 "595-TPD1E04U04DPYR" H 6400 2150 50  0001 C CNN "Mouser"
-F 6 "TPD1E04U04DPYT" H 6400 2150 50  0001 C CNN "Part No"
+F 4 "296-47862-1-ND" H 6400 2150 50  0001 C CNN "DigiKey"
+F 5 "595-TPD1E04U04DPLT" H 6400 2150 50  0001 C CNN "Mouser"
+F 6 "TPD1E04U04DPLT" H 6400 2150 50  0001 C CNN "Part No"
 	1    6400 2150
 	1    0    0    -1
@@
 F 0 "D12" H 6125 4475 50  0000 L CNN
 F 1 "TPD1E04U04" H 6125 4400 50  0000 L CNN
-F 2 "Diode_SMD:D_0201_0603Metric" H 6525 4150 50  0001 C CNN
+F 2 "udriver3:D_0201_0603Metric" H 6525 4150 50  0001 C CNN
 F 3 "https://www.ti.com/lit/ds/symlink/tpd1e04u04.pdf" H 6525 4150 50  0001 C CNN
-F 4 "296-47224-1-ND" H 6425 4150 50  0001 C CNN "DigiKey"
-F 5 "595-TPD1E04U04DPYR" H 6425 4150 50  0001 C CNN "Mouser"
-F 6 "TPD1E04U04DPYT" H 6425 4150 50  0001 C CNN "Part No"
+F 4 "296-47862-1-ND" H 6425 4150 50  0001 C CNN "DigiKey"
+F 5 "595-TPD1E04U04DPLT" H 6425 4150 50  0001 C CNN "Mouser"
+F 6 "TPD1E04U04DPLT" H 6425 4150 50  0001 C CNN "Part No"
 	1    6425 4150
 	1    0    0    -1
@@
 F 0 "D13" H 8250 4450 50  0000 L CNN
 F 1 "TPD1E04U04" H 8250 4375 50  0000 L CNN
-F 2 "Diode_SMD:D_0201_0603Metric" H 8650 4125 50  0001 C CNN
+F 2 "udriver3:D_0201_0603Metric" H 8650 4125 50  0001 C CNN
 F 3 "https://www.ti.com/lit/ds/symlink/tpd1e04u04.pdf" H 8650 4125 50  0001 C CNN
-F 4 "296-47224-1-ND" H 8550 4125 50  0001 C CNN "DigiKey"
-F 5 "595-TPD1E04U04DPYR" H 8550 4125 50  0001 C CNN "Mouser"
-F 6 "TPD1E04U04DPYT" H 8550 4125 50  0001 C CNN "Part No"
+F 4 "296-47862-1-ND" H 8550 4125 50  0001 C CNN "DigiKey"
+F 5 "595-TPD1E04U04DPLT" H 8550 4125 50  0001 C CNN "Mouser"
+F 6 "TPD1E04U04DPLT" H 8550 4125 50  0001 C CNN "Part No"
 	1    8550 4125
 	1    0    0    -1
