File: hardware/udriver3/OMODRI_CAN.kicad_sch (KiCad schematic)
At the start: 4 parts, among them J7 Conn_01x02, U8 TCAN332G

Commit message: Move CAN connector, Include add DC DC back for 1.2 and 3.3V, wire the encoder, ...
Parts:
- J7: footprint udriver3:Hirose_DF13-02P-1.25DSA_1x02_P1.25mm_Vertical -> Connector_Hirose:Hirose_DF13C_CL535-0402-2-51_1x02-1MP_P1.25mm_Vertical
Changed lines of the file:
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@@
       (effects (font (size 1.27 1.27)) (justify left))
     )
-    (property "Footprint" "udriver3:Hirose_DF13-02P-1.25DSA_1x02_P1.25mm_Vertical" (id 2) (at 172.72 91.44 0)
+    (property "Footprint" "Connector_Hirose:Hirose_DF13C_CL535-0402-2-51_1x02-1MP_P1.25mm_Vertical" (id 2) (at 172.72 91.44 0)
       (effects (font (size 1.27 1.27)) hide)
     )

Commit message: Use angle DF13 connector for SPI, CAN and encoders, add 3d step files, route
Parts:
- J7: footprint Connector_Hirose:Hirose_DF13C_CL535-0402-2-51_1x02-1MP_P1.25mm_Vertical -> udriver3:DF13A2P125H21
Changed lines of the file:
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@@
       (effects (font (size 1.27 1.27)) (justify left))
     )
-    (property "Footprint" "Connector_Hirose:Hirose_DF13C_CL535-0402-2-51_1x02-1MP_P1.25mm_Vertical" (id 2) (at 172.72 91.44 0)
+    (property "Footprint" "udriver3:DF13A2P125H21" (id 2) (at 172.72 91.44 0)
       (effects (font (size 1.27 1.27)) hide)
     )

Commit message: minor
Parts:
- J7: footprint udriver3:DF13A2P125H21 -> udriver3:DF132P125H75
Changed lines of the file:
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@@
       (effects (font (size 1.27 1.27)) (justify left))
     )
-    (property "Footprint" "udriver3:DF13A2P125H21" (id 2) (at 172.72 91.44 0)
+    (property "Footprint" "udriver3:DF132P125H75" (id 2) (at 172.72 91.44 0)
       (effects (font (size 1.27 1.27)) hide)
     )

Commit message: Schematics update. 12V0 and 5V0 power supplies not finished yet. RS485 added but not connected to F28388 mcu.
Parts:
- C67: Rated Voltage 10V -> 25V
Changed lines of the file:
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@@
     (title "Open MOtor DRiver Initiative (OMODRI)")
     (date "2020-12-16")
-    (rev "1.1")
+    (rev "2.0")
     (company "LAAS/CNRS")
   )
@@
       (effects (font (size 1.27 1.27)) hide)
     )
-    (property "Rated Voltage" "10V" (id 10) (at 125.73 73.66 0)
+    (property "Rated Voltage" "25V" (id 10) (at 125.73 73.66 0)
       (effects (font (size 1.27 1.27)) hide)
     )

Commit message: Temporary version of udrive3 v2.0. - In schematic there are 2 solutions for DC/DC buck converter. - PCB routing is not finished yet.
Parts:
- removed J7: Conn_01x02, udriver3:DF132P125H75, symbol Connector_Generic:Conn_01x02
- added J7: conn_01x02_MountingPins, udriver3:Hirose_DF13_02P-1.25H_1x02_P1.25mm_Horizontal, symbol omodri_lib:conn_01x02_MountingPins
Connections:
- net CAN_H: now also J7.1 (Pin_1)
- net CAN_L: now also J7.2 (Pin_2)
- net GND: now also J7.MP1 (MountPin1), J7.MP2 (MountPin2)
Changed lines of the file:
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@@
   (junction (at 125.73 69.85) (diameter 0) (color 0 0 0 0)
   )
+  (wire (pts (xy 175.26 99.06) (xy 175.26 102.235))
+    (stroke (width 0) (type default) (color 0 0 0 0))
+  )
   (wire (pts (xy 123.19 69.85) (xy 125.73 69.85))
     (stroke (width 0) (type default) (color 0 0 0 0))
   )
+  (wire (pts (xy 170.18 93.98) (xy 167.64 93.98))
+    (stroke (width 0) (type default) (color 0 0 0 0))
+  )
   (wire (pts (xy 157.48 96.52) (xy 167.64 96.52))
     (stroke (width 0) (type default) (color 0 0 0 0))
   )
+  (wire (pts (xy 167.64 91.44) (xy 170.18 91.44))
+    (stroke (width 0) (type default) (color 0 0 0 0))
+  )
   (wire (pts (xy 118.11 90.17) (xy 121.92 90.17))
     (stroke (width 0) (type default) (color 0 0 0 0))
   )
   (wire (pts (xy 148.59 96.52) (xy 148.59 95.25))
+    (stroke (width 0) (type default) (color 0 0 0 0))
+  )
+  (wire (pts (xy 175.26 86.36) (xy 175.26 83.185))
     (stroke (width 0) (type default) (color 0 0 0 0))
   )
@@
     (pin "2")
   )
-  (symbol (lib_id "Connector_Generic:Conn_01x02") (at 172.72 91.44 0) (unit 1)
-    (in_bom yes) (on_board yes)
-    (property "Reference" "J7" (id 0) (at 174.752 91.6432 0)
-      (effects (font (size 1.27 1.27)) (justify left))
-    )
-    (property "Value" "Conn_01x02" (id 1) (at 174.752 93.9546 0)
-      (effects (font (size 1.27 1.27)) (justify left))
-    )
-    (property "Footprint" "udriver3:DF132P125H75" (id 2) (at 172.72 91.44 0)
-      (effects (font (size 1.27 1.27)) hide)
-    )
-    (property "Datasheet" "~" (id 3) (at 172.72 91.44 0)
-      (effects (font (size 1.27 1.27)) hide)
-    )
-    (property "DigiKey" "H2191-ND" (id 4) (at 172.72 91.44 0)
-      (effects (font (size 1.27 1.27)) hide)
-    )
-    (property "Farnell" "2427585" (id 5) (at 172.72 91.44 0)
-      (effects (font (size 1.27 1.27)) hide)
-    )
-    (property "Mouser" "798-DF13-2P-1.25DSA" (id 6) (at 172.72 91.44 0)
-      (effects (font (size 1.27 1.27)) hide)
-    )
-    (property "Part No" "DF13-2P-1.25DSA" (id 7) (at 172.72 91.44 0)
-      (effects (font (size 1.27 1.27)) hide)
-    )
-    (property "RS" "" (id 8) (at 172.72 91.44 0)
-      (effects (font (size 1.27 1.27)) hide)
-    )
-    (pin "1")
-    (pin "2")
+  (symbol (lib_id "power:GND") (at 175.26 83.185 180) (unit 1)
+    (in_bom yes) (on_board yes)
+    (property "Reference" "#PWR0174" (id 0) (at 175.26 76.835 0)
+      (effects (font (size 1.27 1.27)) hide)
+    )
+    (property "Value" "GND" (id 1) (at 175.133 78.7908 0))
+    (property "Footprint" "" (id 2) (at 175.26 83.185 0)
+      (effects (font (size 1.27 1.27)) hide)
+    )
+    (property "Datasheet" "" (id 3) (at 175.26 83.185 0)
+      (effects (font (size 1.27 1.27)) hide)
+    )
+    (pin "1")
+  )
+  (symbol (lib_id "omodri_lib:conn_01x02_MountingPins") (at 175.26 92.71 0) (unit 1)
+    (in_bom yes) (on_board yes) (fields_autoplaced)
+    (property "Reference" "J7" (id 0) (at 177.292 91.8753 0)
+      (effects (font (size 1.27 1.27)) (justify left))
+    )
+    (property "Value" "conn_01x02_MountingPins" (id 1) (at 177.292 94.4122 0)
+      (effects (font (size 1.27 1.27)) (justify left))
+    )
+    (property "Footprint" "udriver3:Hirose_DF13_02P-1.25H_1x02_P1.25mm_Horizontal" (id 2) (at 175.26 92.71 0)
+      (effects (font (size 1.27 1.27)) hide)
+    )
+    (property "Datasheet" "" (id 3) (at 175.26 92.71 0)
+      (effects (font (size 1.27 1.27)) hide)
+    )
+    (property "DigiKey" "H2191-ND" (id 4) (at 175.26 92.71 0)
+      (effects (font (size 1.27 1.27)) hide)
+    )
+    (property "Farnell" "2427585" (id 5) (at 175.26 92.71 0)
+      (effects (font (size 1.27 1.27)) hide)
+    )
+    (property "Mouser" "798-DF13-2P-1.25DSA" (id 6) (at 175.26 92.71 0)
+      (effects (font (size 1.27 1.27)) hide)
+    )
+    (property "Part No" "DF13-2P-1.25DSA" (id 7) (at 175.26 92.71 0)
+      (effects (font (size 1.27 1.27)) hide)
+    )
+    (property "RS" "H2191-ND" (id 8) (at 175.26 92.71 0)
+      (effects (font (size 1.27 1.27)) hide)
+    )
+    (pin "1")
+    (pin "2")
+    (pin "MP1")
+    (pin "MP2")
+  )
+  (symbol (lib_id "power:GND") (at 175.26 102.235 0) (unit 1)
+    (in_bom yes) (on_board yes)
+    (property "Reference" "#PWR0173" (id 0) (at 175.26 108.585 0)
+      (effects (font (size 1.27 1.27)) hide)
+    )
+    (property "Value" "GND" (id 1) (at 175.387 106.6292 0))
+    (property "Footprint" "" (id 2) (at 175.26 102.235 0)
+      (effects (font (size 1.27 1.27)) hide)
+    )
+    (property "Datasheet" "" (id 3) (at 175.26 102.235 0)
+      (effects (font (size 1.27 1.27)) hide)
+    )
+    (pin "1")
   )
 )
