File: hardware/udriver3/OMODRI_QuadEncod.kicad_sch (KiCad schematic)
At the start: 20 parts, among them J5 conn_01x05_MountingPins, J6 conn_01x05_MountingPins, U21 74LVC2G17, U22 74LVC2G17, U23 74LVC2G17

Commit message: Some routing updates.
Parts:
- J5, J6: DigiKey H2194-ND -> H126405-ND; Farnell 2427589 -> 3019728; Mouser 798-DF13-5P-1.25DSA -> 798-DF13-5P-1.25H76; Part No DF13-5P-1.25DSA -> DF13-5P-1.25H(76); RS 503-7912 -> 188-6306
- U21, U22, U23: DigiKey 296-34875-2-ND -> 1727-7017-2-ND; Mouser 595-SN74LVC2G17DRYR -> 771-LVC2G17GM115; Part No SN74LVC2G17DRYR -> 74LVC2G17GM,115
Changed lines of the file:
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@@
       (effects (font (size 1.27 1.27)) hide)
     )
-    (property "DigiKey" "296-34875-2-ND" (id 4) (at 210.82 121.92 0)
-      (effects (font (size 1.27 1.27)) hide)
-    )
-    (property "Mouser" "595-SN74LVC2G17DRYR" (id 5) (at 210.82 121.92 0)
-      (effects (font (size 1.27 1.27)) hide)
-    )
-    (property "Part No" "SN74LVC2G17DRYR" (id 6) (at 210.82 121.92 0)
+    (property "DigiKey" "1727-7017-2-ND" (id 4) (at 210.82 121.92 0)
+      (effects (font (size 1.27 1.27)) hide)
+    )
+    (property "Mouser" "771-LVC2G17GM115" (id 5) (at 210.82 121.92 0)
+      (effects (font (size 1.27 1.27)) hide)
+    )
+    (property "Part No" "74LVC2G17GM,115" (id 6) (at 210.82 121.92 0)
       (effects (font (size 1.27 1.27)) hide)
     )
@@
       (effects (font (size 1.27 1.27)) hide)
     )
-    (property "DigiKey" "H2194-ND" (id 4) (at 83.82 110.49 0)
-      (effects (font (size 1.27 1.27)) hide)
-    )
-    (property "Farnell" "2427589" (id 5) (at 83.82 110.49 0)
-      (effects (font (size 1.27 1.27)) hide)
-    )
-    (property "Mouser" "798-DF13-5P-1.25DSA" (id 6) (at 83.82 110.49 0)
-      (effects (font (size 1.27 1.27)) hide)
-    )
-    (property "Part No" "DF13-5P-1.25DSA" (id 7) (at 83.82 110.49 0)
-      (effects (font (size 1.27 1.27)) hide)
-    )
-    (property "RS" "503-7912" (id 8) (at 83.82 110.49 0)
+    (property "DigiKey" "H126405-ND" (id 4) (at 83.82 110.49 0)
+      (effects (font (size 1.27 1.27)) hide)
+    )
+    (property "Farnell" "3019728" (id 5) (at 83.82 110.49 0)
+      (effects (font (size 1.27 1.27)) hide)
+    )
+    (property "Mouser" "798-DF13-5P-1.25H76" (id 6) (at 83.82 110.49 0)
+      (effects (font (size 1.27 1.27)) hide)
+    )
+    (property "Part No" "DF13-5P-1.25H(76)" (id 7) (at 83.82 110.49 0)
+      (effects (font (size 1.27 1.27)) hide)
+    )
+    (property "RS" "188-6306" (id 8) (at 83.82 110.49 0)
       (effects (font (size 1.27 1.27)) hide)
     )
@@
       (effects (font (size 1.27 1.27)) hide)
     )
-    (property "DigiKey" "296-34875-2-ND" (id 4) (at 165.1 58.42 0)
-      (effects (font (size 1.27 1.27)) hide)
-    )
-    (property "Mouser" "595-SN74LVC2G17DRYR" (id 5) (at 165.1 58.42 0)
-      (effects (font (size 1.27 1.27)) hide)
-    )
-    (property "Part No" "SN74LVC2G17DRYR" (id 6) (at 165.1 58.42 0)
+    (property "DigiKey" "1727-7017-2-ND" (id 4) (at 165.1 58.42 0)
+      (effects (font (size 1.27 1.27)) hide)
+    )
+    (property "Mouser" "771-LVC2G17GM115" (id 5) (at 165.1 58.42 0)
+      (effects (font (size 1.27 1.27)) hide)
+    )
+    (property "Part No" "74LVC2G17GM,115" (id 6) (at 165.1 58.42 0)
       (effects (font (size 1.27 1.27)) hide)
     )
@@
       (effects (font (size 1.27 1.27)) hide)
     )
-    (property "DigiKey" "296-34875-2-ND" (id 4) (at 210.82 58.42 0)
-      (effects (font (size 1.27 1.27)) hide)
-    )
-    (property "Mouser" "595-SN74LVC2G17DRYR" (id 5) (at 210.82 58.42 0)
-      (effects (font (size 1.27 1.27)) hide)
-    )
-    (property "Part No" "SN74LVC2G17DRYR" (id 6) (at 210.82 58.42 0)
+    (property "DigiKey" "1727-7017-2-ND" (id 4) (at 210.82 58.42 0)
+      (effects (font (size 1.27 1.27)) hide)
+    )
+    (property "Mouser" "771-LVC2G17GM115" (id 5) (at 210.82 58.42 0)
+      (effects (font (size 1.27 1.27)) hide)
+    )
+    (property "Part No" "74LVC2G17GM,115" (id 6) (at 210.82 58.42 0)
       (effects (font (size 1.27 1.27)) hide)
     )
@@
       (effects (font (size 1.27 1.27)) hide)
     )
-    (property "DigiKey" "296-34875-2-ND" (id 4) (at 165.1 121.92 0)
-      (effects (font (size 1.27 1.27)) hide)
-    )
-    (property "Mouser" "595-SN74LVC2G17DRYR" (id 5) (at 165.1 121.92 0)
-      (effects (font (size 1.27 1.27)) hide)
-    )
-    (property "Part No" "SN74LVC2G17DRYR" (id 6) (at 165.1 121.92 0)
+    (property "DigiKey" "1727-7017-2-ND" (id 4) (at 165.1 121.92 0)
+      (effects (font (size 1.27 1.27)) hide)
+    )
+    (property "Mouser" "771-LVC2G17GM115" (id 5) (at 165.1 121.92 0)
+      (effects (font (size 1.27 1.27)) hide)
+    )
+    (property "Part No" "74LVC2G17GM,115" (id 6) (at 165.1 121.92 0)
       (effects (font (size 1.27 1.27)) hide)
     )
@@
       (effects (font (size 1.27 1.27)) hide)
     )
-    (property "DigiKey" "H2194-ND" (id 4) (at 83.82 58.42 0)
-      (effects (font (size 1.27 1.27)) hide)
-    )
-    (property "Farnell" "2427589" (id 5) (at 83.82 58.42 0)
-      (effects (font (size 1.27 1.27)) hide)
-    )
-    (property "Mouser" "798-DF13-5P-1.25DSA" (id 6) (at 83.82 58.42 0)
-      (effects (font (size 1.27 1.27)) hide)
-    )
-    (property "Part No" "DF13-5P-1.25DSA" (id 7) (at 83.82 58.42 0)
-      (effects (font (size 1.27 1.27)) hide)
-    )
-    (property "RS" "503-7912" (id 8) (at 83.82 58.42 0)
+    (property "DigiKey" "H126405-ND" (id 4) (at 83.82 58.42 0)
+      (effects (font (size 1.27 1.27)) hide)
+    )
+    (property "Farnell" "3019728" (id 5) (at 83.82 58.42 0)
+      (effects (font (size 1.27 1.27)) hide)
+    )
+    (property "Mouser" "798-DF13-5P-1.25H76" (id 6) (at 83.82 58.42 0)
+      (effects (font (size 1.27 1.27)) hide)
+    )
+    (property "Part No" "DF13-5P-1.25H(76)" (id 7) (at 83.82 58.42 0)
+      (effects (font (size 1.27 1.27)) hide)
+    )
+    (property "RS" "188-6306" (id 8) (at 83.82 58.42 0)
       (effects (font (size 1.27 1.27)) hide)
     )
@@
       (effects (font (size 1.27 1.27)) hide)
     )
-    (property "DigiKey" "296-34875-2-ND" (id 4) (at 165.1 90.17 0)
-      (effects (font (size 1.27 1.27)) hide)
-    )
-    (property "Mouser" "595-SN74LVC2G17DRYR" (id 5) (at 165.1 90.17 0)
-      (effects (font (size 1.27 1.27)) hide)
-    )
-    (property "Part No" "SN74LVC2G17DRYR" (id 6) (at 165.1 90.17 0)
+    (property "DigiKey" "1727-7017-2-ND" (id 4) (at 165.1 90.17 0)
+      (effects (font (size 1.27 1.27)) hide)
+    )
+    (property "Mouser" "771-LVC2G17GM115" (id 5) (at 165.1 90.17 0)
+      (effects (font (size 1.27 1.27)) hide)
+    )
+    (property "Part No" "74LVC2G17GM,115" (id 6) (at 165.1 90.17 0)
       (effects (font (size 1.27 1.27)) hide)
     )
@@
       (effects (font (size 1.27 1.27)) hide)
     )
-    (property "DigiKey" "296-34875-2-ND" (id 4) (at 210.82 90.17 0)
-      (effects (font (size 1.27 1.27)) hide)
-    )
-    (property "Mouser" "595-SN74LVC2G17DRYR" (id 5) (at 210.82 90.17 0)
-      (effects (font (size 1.27 1.27)) hide)
-    )
-    (property "Part No" "SN74LVC2G17DRYR" (id 6) (at 210.82 90.17 0)
-      (effects (font (size 1.27 1.27)) hide)
-    )
+    (property "DigiKey" "1727-7017-2-ND" (id 4) (at 210.82 90.17 0)
+      (effects (font (size 1.27 1.27)) hide)
+    )
+    (property "Mouser" "771-LVC2G17GM115" (id 5) (at 210.82 90.17 0)
+      (effects (font (size 1.27 1.27)) hide)
+    )
+    (property "Part No" "74LVC2G17GM,115" (id 6) (at 210.82 90.17 0)
+      (effects (font (size 1.27 1.27)) hide)
+    )
