File: hardware/udriver3/OMODRI_Alim_12V.kicad_sch (KiCad schematic)
At the start: 7 parts, among them U9 TPSM560R6H

Commit message: PCB update. Re-annotation of the design + via stitching (GND).
Parts:
- renumbered C24 to C96, C70 to C97, C31 to C98, C88 to C99, R66 to R58, R67 to R59, U9 to U16
Changed lines of the file:
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@@
   (symbol (lib_id "power:GND") (at 184.15 114.3 0) (unit 1)
     (in_bom yes) (on_board yes)
-    (property "Reference" "#PWR0116" (id 0) (at 184.15 120.65 0)
+    (property "Reference" "#PWR0157" (id 0) (at 184.15 120.65 0)
       (effects (font (size 1.27 1.27)) hide)
     )
@@
   (symbol (lib_id "omodri_lib:TPSM560R6H") (at 137.16 91.44 0) (unit 1)
     (in_bom yes) (on_board yes)
-    (property "Reference" "U9" (id 0) (at 137.16 81.28 0))
+    (property "Reference" "U16" (id 0) (at 137.16 81.28 0))
     (property "Value" "TPSM560R6H" (id 1) (at 137.16 83.82 0))
     (property "Footprint" "udriver3:B3QFN_15" (id 2) (at 137.16 91.44 0)
@@
   (symbol (lib_id "power:GND") (at 91.44 114.3 0) (unit 1)
     (in_bom yes) (on_board yes)
-    (property "Reference" "#PWR060" (id 0) (at 91.44 120.65 0)
+    (property "Reference" "#PWR0151" (id 0) (at 91.44 120.65 0)
       (effects (font (size 1.27 1.27)) hide)
     )
@@
   (symbol (lib_id "Device:C") (at 91.44 100.33 0) (unit 1)
     (in_bom yes) (on_board yes)
-    (property "Reference" "C24" (id 0) (at 93.98 99.06 0)
+    (property "Reference" "C96" (id 0) (at 93.98 99.06 0)
       (effects (font (size 1.27 1.27)) (justify left))
     )
@@
   (symbol (lib_id "power:GND") (at 120.65 114.3 0) (unit 1)
     (in_bom yes) (on_board yes)
-    (property "Reference" "#PWR0119" (id 0) (at 120.65 120.65 0)
+    (property "Reference" "#PWR0154" (id 0) (at 120.65 120.65 0)
       (effects (font (size 1.27 1.27)) hide)
     )
@@
   (symbol (lib_id "power:GND") (at 175.26 114.3 0) (unit 1)
     (in_bom yes) (on_board yes)
-    (property "Reference" "#PWR0115" (id 0) (at 175.26 120.65 0)
+    (property "Reference" "#PWR0156" (id 0) (at 175.26 120.65 0)
       (effects (font (size 1.27 1.27)) hide)
     )
@@
   (symbol (lib_id "Device:R") (at 175.26 107.95 180) (unit 1)
     (in_bom yes) (on_board yes)
-    (property "Reference" "R67" (id 0) (at 180.34 106.68 0)
+    (property "Reference" "R59" (id 0) (at 180.34 106.68 0)
       (effects (font (size 1.27 1.27)) (justify left))
     )
@@
   (symbol (lib_id "Device:C") (at 101.6 100.33 0) (unit 1)
     (in_bom yes) (on_board yes)
-    (property "Reference" "C70" (id 0) (at 104.14 99.06 0)
+    (property "Reference" "C97" (id 0) (at 104.14 99.06 0)
       (effects (font (size 1.27 1.27)) (justify left))
     )
@@
   (symbol (lib_id "Device:R") (at 175.26 91.44 0) (unit 1)
     (in_bom yes) (on_board yes)
-    (property "Reference" "R66" (id 0) (at 177.038 90.2716 0)
+    (property "Reference" "R58" (id 0) (at 177.038 90.2716 0)
       (effects (font (size 1.27 1.27)) (justify left))
     )
@@
   (symbol (lib_id "Device:C") (at 111.76 100.33 0) (unit 1)
     (in_bom yes) (on_board yes)
-    (property "Reference" "C31" (id 0) (at 114.3 99.06 0)
+    (property "Reference" "C98" (id 0) (at 114.3 99.06 0)
       (effects (font (size 1.27 1.27)) (justify left))
     )
@@
   (symbol (lib_id "Device:C") (at 184.15 100.33 0) (unit 1)
     (in_bom yes) (on_board yes)
-    (property "Reference" "C88" (id 0) (at 187.071 99.1616 0)
+    (property "Reference" "C99" (id 0) (at 187.071 99.1616 0)
       (effects (font (size 1.27 1.27)) (justify left))
     )
@@
   (symbol (lib_id "power:GND") (at 101.6 114.3 0) (unit 1)
     (in_bom yes) (on_board yes)
-    (property "Reference" "#PWR0133" (id 0) (at 101.6 120.65 0)
+    (property "Reference" "#PWR0152" (id 0) (at 101.6 120.65 0)
       (effects (font (size 1.27 1.27)) hide)
     )
@@
   (symbol (lib_id "power:GND") (at 161.29 114.3 0) (unit 1)
     (in_bom yes) (on_board yes)
-    (property "Reference" "#PWR0113" (id 0) (at 161.29 120.65 0)
+    (property "Reference" "#PWR0155" (id 0) (at 161.29 120.65 0)
       (effects (font (size 1.27 1.27)) hide)
     )
@@
   (symbol (lib_id "power:GND") (at 111.76 114.3 0) (unit 1)
     (in_bom yes) (on_board yes)
-    (property "Reference" "#PWR0141" (id 0) (at 111.76 120.65 0)
-      (effects (font (size 1.27 1.27)) hide)
-    )
+    (property "Reference" "#PWR0153" (id 0) (at 111.76 120.65 0)
+      (effects (font (size 1.27 1.27)) hide)
+    )

Commit message: PCB updates. - Replace CAN/RS485 120ohm resistor - Replace resistor on TCAN RXD pin - Update of some references - Add some 3D missing models
Parts:
- R58: value 100k -> 10k; DigiKey P122655CT-ND -> P122414CT-ND; Farnell 2302389 -> 2302362; Mouser 667-ERJ-1GNF1003C -> 667-ERJ-1GNF1002C; Part No ERJ-1GNF1003C -> ERJ-1GNF1002C; RS 179-7130 -> 176-3597
- R59: value 9.09k -> 909; DigiKey P122907TR-ND -> P123194TR-ND; Farnell 3335262 -> 3303125; Mouser 667-ERJ-1GNF2941C -> 667-ERJ-1GNF9090C; Part No ERJ-1GNF2941C -> ERJ-1GNF9090C
Changed lines of the file:
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@@
       (effects (font (size 1.27 1.27)) (justify left))
     )
-    (property "Value" "9.09k" (id 1) (at 181.61 109.22 0)
+    (property "Value" "909" (id 1) (at 181.61 109.22 0)
       (effects (font (size 1.27 1.27)) (justify left))
     )
@@
       (effects (font (size 1.27 1.27)) hide)
     )
-    (property "DigiKey" "P122907TR-ND" (id 4) (at 175.26 107.95 0)
+    (property "DigiKey" "P123194TR-ND" (id 4) (at 175.26 107.95 0)
       (effects (font (size 1.27 1.27)) hide)
     )
-    (property "Farnell" "3335262" (id 5) (at 175.26 107.95 0)
+    (property "Farnell" "3303125" (id 5) (at 175.26 107.95 0)
       (effects (font (size 1.27 1.27)) hide)
     )
-    (property "Mouser" "667-ERJ-1GNF2941C" (id 6) (at 175.26 107.95 0)
+    (property "Mouser" "667-ERJ-1GNF9090C" (id 6) (at 175.26 107.95 0)
       (effects (font (size 1.27 1.27)) hide)
     )
-    (property "Part No" "ERJ-1GNF2941C" (id 7) (at 175.26 107.95 0)
+    (property "Part No" "ERJ-1GNF9090C" (id 7) (at 175.26 107.95 0)
       (effects (font (size 1.27 1.27)) hide)
     )
@@
       (effects (font (size 1.27 1.27)) (justify left))
     )
-    (property "Value" "100k" (id 1) (at 177.038 92.583 0)
+    (property "Value" "10k" (id 1) (at 177.038 92.583 0)
       (effects (font (size 1.27 1.27)) (justify left))
     )
@@
       (effects (font (size 1.27 1.27)) hide)
     )
-    (property "DigiKey" "P122655CT-ND" (id 4) (at 175.26 91.44 0)
+    (property "DigiKey" "P122414CT-ND" (id 4) (at 175.26 91.44 0)
       (effects (font (size 1.27 1.27)) hide)
     )
-    (property "Farnell" "2302389" (id 5) (at 175.26 91.44 0)
+    (property "Farnell" "2302362" (id 5) (at 175.26 91.44 0)
       (effects (font (size 1.27 1.27)) hide)
     )
-    (property "Mouser" "667-ERJ-1GNF1003C" (id 6) (at 175.26 91.44 0)
+    (property "Mouser" "667-ERJ-1GNF1002C" (id 6) (at 175.26 91.44 0)
       (effects (font (size 1.27 1.27)) hide)
     )
-    (property "Part No" "ERJ-1GNF1003C" (id 7) (at 175.26 91.44 0)
+    (property "Part No" "ERJ-1GNF1002C" (id 7) (at 175.26 91.44 0)
       (effects (font (size 1.27 1.27)) hide)
     )
-    (property "RS" "179-7130" (id 8) (at 175.26 91.44 0)
+    (property "RS" "176-3597" (id 8) (at 175.26 91.44 0)
       (effects (font (size 1.27 1.27)) hide)
     )
