File: hardware/udriver3/OMODRI_Alim_5V.kicad_sch (KiCad schematic)
At the start: 8 parts, among them U7 TPSM561R5

Commit message: PCB fully routed. Some optimizations need to be done + revue of the schematics.
Connections:
- net PG_12V0 is gone; now on net VPOWER: U7.2 (EN)
- net GND: now also U7.13 (NC4), U7.3 (NC1), U7.6 (NC3)
Changed lines of the file:
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@@
   (junction (at 179.07 92.71) (diameter 0) (color 0 0 0 0)
   )
+  (junction (at 124.46 106.68) (diameter 0) (color 0 0 0 0)
+  )
   (junction (at 165.1 95.25) (diameter 0) (color 0 0 0 0)
   )
   (junction (at 88.9 82.55) (diameter 0) (color 0 0 0 0)
   )
+  (junction (at 124.46 109.22) (diameter 0) (color 0 0 0 0)
+  )
   (junction (at 187.96 82.55) (diameter 0) (color 0 0 0 0)
   )
   (junction (at 124.46 82.55) (diameter 0) (color 0 0 0 0)
   )
+  (junction (at 124.46 85.09) (diameter 0) (color 0 0 0 0)
+  )
   (junction (at 99.06 82.55) (diameter 0) (color 0 0 0 0)
   )
@@
     (stroke (width 0) (type default) (color 0 0 0 0))
   )
+  (wire (pts (xy 124.46 106.68) (xy 132.08 106.68))
+    (stroke (width 0) (type default) (color 0 0 0 0))
+  )
   (wire (pts (xy 153.67 82.55) (xy 158.75 82.55))
     (stroke (width 0) (type default) (color 0 0 0 0))
@@
     (stroke (width 0) (type default) (color 0 0 0 0))
   )
+  (wire (pts (xy 124.46 109.22) (xy 124.46 110.49))
+    (stroke (width 0) (type default) (color 0 0 0 0))
+  )
+  (wire (pts (xy 124.46 101.6) (xy 124.46 106.68))
+    (stroke (width 0) (type default) (color 0 0 0 0))
+  )
+  (wire (pts (xy 124.46 106.68) (xy 124.46 109.22))
+    (stroke (width 0) (type default) (color 0 0 0 0))
+  )
   (wire (pts (xy 187.96 82.55) (xy 187.96 92.71))
     (stroke (width 0) (type default) (color 0 0 0 0))
@@
     (stroke (width 0) (type default) (color 0 0 0 0))
   )
+  (wire (pts (xy 124.46 95.25) (xy 124.46 85.09))
+    (stroke (width 0) (type default) (color 0 0 0 0))
+  )
   (wire (pts (xy 153.67 109.22) (xy 165.1 109.22))
     (stroke (width 0) (type default) (color 0 0 0 0))
@@
     (stroke (width 0) (type default) (color 0 0 0 0))
   )
+  (wire (pts (xy 132.08 101.6) (xy 124.46 101.6))
+    (stroke (width 0) (type default) (color 0 0 0 0))
+  )
   (wire (pts (xy 179.07 82.55) (xy 179.07 83.82))
     (stroke (width 0) (type default) (color 0 0 0 0))
@@
     (stroke (width 0) (type default) (color 0 0 0 0))
   )
-  (wire (pts (xy 127 95.25) (xy 128.27 95.25))
+  (wire (pts (xy 124.46 109.22) (xy 132.08 109.22))
+    (stroke (width 0) (type default) (color 0 0 0 0))
+  )
+  (wire (pts (xy 124.46 95.25) (xy 128.27 95.25))
     (stroke (width 0) (type default) (color 0 0 0 0))
   )
@@
   (hierarchical_label "PG_5V0" (shape output) (at 167.64 95.25 0)
     (effects (font (size 1.27 1.27)) (justify left))
-  )
-  (hierarchical_label "PG_12V0" (shape input) (at 127 95.25 180)
-    (effects (font (size 1.27 1.27)) (justify right))
   )
   (symbol (lib_id "power:GND") (at 99.06 110.49 0) (unit 1)
@@
     (pin "2")
   )
+  (symbol (lib_id "power:GND") (at 124.46 110.49 0) (unit 1)
+    (in_bom yes) (on_board yes)
+    (property "Reference" "#PWR0118" (id 0) (at 124.46 116.84 0)
+      (effects (font (size 1.27 1.27)) hide)
+    )
+    (property "Value" "GND" (id 1) (at 124.587 114.8842 0))
+    (property "Footprint" "" (id 2) (at 124.46 110.49 0)
+      (effects (font (size 1.27 1.27)) hide)
+    )
+    (property "Datasheet" "" (id 3) (at 124.46 110.49 0)
+      (effects (font (size 1.27 1.27)) hide)
+    )
+    (pin "1")
+  )
   (symbol (lib_id "power:GND") (at 165.1 110.49 0) (unit 1)

Commit message: PCB update. Re-annotation of the design + via stitching (GND).
Parts:
- renumbered C89 to C57, C60 to C58, C62 to C59, C66 to C60, R53 to R49, R57 to R50, R59 to R51, U7 to U12
Changed lines of the file:
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@@
   (symbol (lib_id "power:GND") (at 99.06 110.49 0) (unit 1)
     (in_bom yes) (on_board yes)
-    (property "Reference" "#PWR0105" (id 0) (at 99.06 116.84 0)
+    (property "Reference" "#PWR0125" (id 0) (at 99.06 116.84 0)
       (effects (font (size 1.27 1.27)) hide)
     )
@@
   (symbol (lib_id "Device:C") (at 88.9 96.52 0) (unit 1)
     (in_bom yes) (on_board yes)
-    (property "Reference" "C89" (id 0) (at 91.44 95.25 0)
+    (property "Reference" "C57" (id 0) (at 91.44 95.25 0)
       (effects (font (size 1.27 1.27)) (justify left))
     )
@@
   (symbol (lib_id "Device:C") (at 99.06 96.52 0) (unit 1)
     (in_bom yes) (on_board yes)
-    (property "Reference" "C60" (id 0) (at 101.6 95.25 0)
+    (property "Reference" "C58" (id 0) (at 101.6 95.25 0)
       (effects (font (size 1.27 1.27)) (justify left))
     )
@@
   (symbol (lib_id "power:GND") (at 88.9 110.49 0) (unit 1)
     (in_bom yes) (on_board yes)
-    (property "Reference" "#PWR049" (id 0) (at 88.9 116.84 0)
+    (property "Reference" "#PWR0124" (id 0) (at 88.9 116.84 0)
       (effects (font (size 1.27 1.27)) hide)
     )
@@
   (symbol (lib_id "power:GND") (at 109.22 110.49 0) (unit 1)
     (in_bom yes) (on_board yes)
-    (property "Reference" "#PWR0112" (id 0) (at 109.22 116.84 0)
+    (property "Reference" "#PWR0126" (id 0) (at 109.22 116.84 0)
       (effects (font (size 1.27 1.27)) hide)
     )
@@
   (symbol (lib_id "power:GND") (at 179.07 110.49 0) (unit 1)
     (in_bom yes) (on_board yes)
-    (property "Reference" "#PWR0130" (id 0) (at 179.07 116.84 0)
+    (property "Reference" "#PWR0129" (id 0) (at 179.07 116.84 0)
       (effects (font (size 1.27 1.27)) hide)
     )
@@
   (symbol (lib_id "omodri_lib:TPSM561R5") (at 140.97 87.63 0) (unit 1)
     (in_bom yes) (on_board yes)
-    (property "Reference" "U7" (id 0) (at 140.97 77.47 0))
+    (property "Reference" "U12" (id 0) (at 140.97 77.47 0))
     (property "Value" "TPSM561R5" (id 1) (at 140.97 80.01 0))
     (property "Footprint" "udriver3:B3QFN_15" (id 2) (at 140.97 87.63 0)
@@
   (symbol (lib_id "Device:C") (at 109.22 96.52 0) (unit 1)
     (in_bom yes) (on_board yes)
-    (property "Reference" "C62" (id 0) (at 111.76 95.25 0)
+    (property "Reference" "C59" (id 0) (at 111.76 95.25 0)
       (effects (font (size 1.27 1.27)) (justify left))
     )
@@
   (symbol (lib_id "Device:C") (at 187.96 96.52 0) (unit 1)
     (in_bom yes) (on_board yes)
-    (property "Reference" "C66" (id 0) (at 190.881 95.3516 0)
+    (property "Reference" "C60" (id 0) (at 190.881 95.3516 0)
       (effects (font (size 1.27 1.27)) (justify left))
     )
@@
   (symbol (lib_id "Device:R") (at 179.07 104.14 180) (unit 1)
     (in_bom yes) (on_board yes)
-    (property "Reference" "R59" (id 0) (at 184.15 102.87 0)
+    (property "Reference" "R51" (id 0) (at 184.15 102.87 0)
       (effects (font (size 1.27 1.27)) (justify left))
     )
@@
   (symbol (lib_id "power:GND") (at 124.46 110.49 0) (unit 1)
     (in_bom yes) (on_board yes)
-    (property "Reference" "#PWR0118" (id 0) (at 124.46 116.84 0)
+    (property "Reference" "#PWR0127" (id 0) (at 124.46 116.84 0)
       (effects (font (size 1.27 1.27)) hide)
     )
@@
   (symbol (lib_id "power:GND") (at 165.1 110.49 0) (unit 1)
     (in_bom yes) (on_board yes)
-    (property "Reference" "#PWR0129" (id 0) (at 165.1 116.84 0)
+    (property "Reference" "#PWR0128" (id 0) (at 165.1 116.84 0)
       (effects (font (size 1.27 1.27)) hide)
     )
@@
   (symbol (lib_id "power:GND") (at 187.96 110.49 0) (unit 1)
     (in_bom yes) (on_board yes)
-    (property "Reference" "#PWR0132" (id 0) (at 187.96 116.84 0)
+    (property "Reference" "#PWR0130" (id 0) (at 187.96 116.84 0)
       (effects (font (size 1.27 1.27)) hide)
     )
@@
   (symbol (lib_id "Device:R") (at 179.07 87.63 0) (unit 1)
     (in_bom yes) (on_board yes)
-    (property "Reference" "R53" (id 0) (at 180.848 86.4616 0)
+    (property "Reference" "R49" (id 0) (at 180.848 86.4616 0)
       (effects (font (size 1.27 1.27)) (justify left))
     )
@@
   (symbol (lib_id "Device:R") (at 165.1 99.06 0) (unit 1)
     (in_bom yes) (on_board yes)
-    (property "Reference" "R57" (id 0) (at 166.878 97.8916 0)
-      (effects (font (size 1.27 1.27)) (justify left))
-    )
+    (property "Reference" "R50" (id 0) (at 166.878 97.8916 0)
+      (effects (font (size 1.27 1.27)) (justify left))
+    )

Commit message: PCB updates. - Replace CAN/RS485 120ohm resistor - Replace resistor on TCAN RXD pin - Update of some references - Add some 3D missing models
Parts:
- R49: value 100k -> 10k; DigiKey P122655CT-ND -> P122414CT-ND; Farnell 2302389 -> 2302362; Mouser 667-ERJ-1GNF1003C -> 667-ERJ-1GNF1002C; Part No ERJ-1GNF1003C -> ERJ-1GNF1002C; RS 179-7130 -> 176-3597
Changed lines of the file:
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@@
       (effects (font (size 1.27 1.27)) (justify left))
     )
-    (property "Value" "100k" (id 1) (at 180.848 88.773 0)
+    (property "Value" "10k" (id 1) (at 180.848 88.773 0)
       (effects (font (size 1.27 1.27)) (justify left))
     )
@@
       (effects (font (size 1.27 1.27)) hide)
     )
-    (property "DigiKey" "P122655CT-ND" (id 4) (at 179.07 87.63 0)
+    (property "DigiKey" "P122414CT-ND" (id 4) (at 179.07 87.63 0)
       (effects (font (size 1.27 1.27)) hide)
     )
-    (property "Farnell" "2302389" (id 5) (at 179.07 87.63 0)
+    (property "Farnell" "2302362" (id 5) (at 179.07 87.63 0)
       (effects (font (size 1.27 1.27)) hide)
     )
-    (property "Mouser" "667-ERJ-1GNF1003C" (id 6) (at 179.07 87.63 0)
+    (property "Mouser" "667-ERJ-1GNF1002C" (id 6) (at 179.07 87.63 0)
       (effects (font (size 1.27 1.27)) hide)
     )
-    (property "Part No" "ERJ-1GNF1003C" (id 7) (at 179.07 87.63 0)
+    (property "Part No" "ERJ-1GNF1002C" (id 7) (at 179.07 87.63 0)
       (effects (font (size 1.27 1.27)) hide)
     )
-    (property "RS" "179-7130" (id 8) (at 179.07 87.63 0)
+    (property "RS" "176-3597" (id 8) (at 179.07 87.63 0)
       (effects (font (size 1.27 1.27)) hide)
     )

Commit message: PCB updates - FSI protection added against FPC cable reverse connection - BOSCH BMI088 IMU added.
Parts:
- renumbered C57 to C58, C58 to C59, C59 to C60, C60 to C61, R49 to R50, R50 to R51, R51 to R52
Changed lines of the file:
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@@
   (title_block
     (title "Open MOtor DRiver Initiative (OMODRI)")
-    (date "2022-10-05")
+    (date "2022-11-24")
     (rev "2.0")
     (company "LAAS/CNRS")
@@
   (symbol (lib_id "power:GND") (at 99.06 110.49 0) (unit 1)
     (in_bom yes) (on_board yes)
-    (property "Reference" "#PWR0125" (id 0) (at 99.06 116.84 0)
+    (property "Reference" "#PWR0126" (id 0) (at 99.06 116.84 0)
       (effects (font (size 1.27 1.27)) hide)
     )
@@
   (symbol (lib_id "Device:C") (at 88.9 96.52 0) (unit 1)
     (in_bom yes) (on_board yes)
-    (property "Reference" "C57" (id 0) (at 91.44 95.25 0)
+    (property "Reference" "C58" (id 0) (at 91.44 95.25 0)
       (effects (font (size 1.27 1.27)) (justify left))
     )
@@
   (symbol (lib_id "Device:C") (at 99.06 96.52 0) (unit 1)
     (in_bom yes) (on_board yes)
-    (property "Reference" "C58" (id 0) (at 101.6 95.25 0)
+    (property "Reference" "C59" (id 0) (at 101.6 95.25 0)
       (effects (font (size 1.27 1.27)) (justify left))
     )
@@
   (symbol (lib_id "power:GND") (at 88.9 110.49 0) (unit 1)
     (in_bom yes) (on_board yes)
-    (property "Reference" "#PWR0124" (id 0) (at 88.9 116.84 0)
+    (property "Reference" "#PWR0125" (id 0) (at 88.9 116.84 0)
       (effects (font (size 1.27 1.27)) hide)
     )
@@
   (symbol (lib_id "power:GND") (at 109.22 110.49 0) (unit 1)
     (in_bom yes) (on_board yes)
-    (property "Reference" "#PWR0126" (id 0) (at 109.22 116.84 0)
+    (property "Reference" "#PWR0127" (id 0) (at 109.22 116.84 0)
       (effects (font (size 1.27 1.27)) hide)
     )
@@
   (symbol (lib_id "power:GND") (at 179.07 110.49 0) (unit 1)
     (in_bom yes) (on_board yes)
-    (property "Reference" "#PWR0129" (id 0) (at 179.07 116.84 0)
+    (property "Reference" "#PWR0130" (id 0) (at 179.07 116.84 0)
       (effects (font (size 1.27 1.27)) hide)
     )
@@
   (symbol (lib_id "Device:C") (at 109.22 96.52 0) (unit 1)
     (in_bom yes) (on_board yes)
-    (property "Reference" "C59" (id 0) (at 111.76 95.25 0)
+    (property "Reference" "C60" (id 0) (at 111.76 95.25 0)
       (effects (font (size 1.27 1.27)) (justify left))
     )
@@
   (symbol (lib_id "Device:C") (at 187.96 96.52 0) (unit 1)
     (in_bom yes) (on_board yes)
-    (property "Reference" "C60" (id 0) (at 190.881 95.3516 0)
+    (property "Reference" "C61" (id 0) (at 190.881 95.3516 0)
       (effects (font (size 1.27 1.27)) (justify left))
     )
@@
   (symbol (lib_id "Device:R") (at 179.07 104.14 180) (unit 1)
     (in_bom yes) (on_board yes)
-    (property "Reference" "R51" (id 0) (at 184.15 102.87 0)
+    (property "Reference" "R52" (id 0) (at 184.15 102.87 0)
       (effects (font (size 1.27 1.27)) (justify left))
     )
@@
   (symbol (lib_id "power:GND") (at 124.46 110.49 0) (unit 1)
     (in_bom yes) (on_board yes)
-    (property "Reference" "#PWR0127" (id 0) (at 124.46 116.84 0)
+    (property "Reference" "#PWR0128" (id 0) (at 124.46 116.84 0)
       (effects (font (size 1.27 1.27)) hide)
     )
@@
   (symbol (lib_id "power:GND") (at 165.1 110.49 0) (unit 1)
     (in_bom yes) (on_board yes)
-    (property "Reference" "#PWR0128" (id 0) (at 165.1 116.84 0)
+    (property "Reference" "#PWR0129" (id 0) (at 165.1 116.84 0)
       (effects (font (size 1.27 1.27)) hide)
     )
@@
   (symbol (lib_id "power:GND") (at 187.96 110.49 0) (unit 1)
     (in_bom yes) (on_board yes)
-    (property "Reference" "#PWR0130" (id 0) (at 187.96 116.84 0)
+    (property "Reference" "#PWR0131" (id 0) (at 187.96 116.84 0)
       (effects (font (size 1.27 1.27)) hide)
     )
@@
   (symbol (lib_id "Device:R") (at 179.07 87.63 0) (unit 1)
     (in_bom yes) (on_board yes)
-    (property "Reference" "R49" (id 0) (at 180.848 86.4616 0)
+    (property "Reference" "R50" (id 0) (at 180.848 86.4616 0)
       (effects (font (size 1.27 1.27)) (justify left))
     )
@@
   (symbol (lib_id "Device:R") (at 165.1 99.06 0) (unit 1)
     (in_bom yes) (on_board yes)
-    (property "Reference" "R50" (id 0) (at 166.878 97.8916 0)
-      (effects (font (size 1.27 1.27)) (justify left))
-    )
+    (property "Reference" "R51" (id 0) (at 166.878 97.8916 0)
+      (effects (font (size 1.27 1.27)) (justify left))
+    )

Commit message: PCB udpates. - add serial resistors on boot jumpers - modify config jumpers to be opened by default
Parts:
- renumbered C58 to C56, C59 to C57, C60 to C58, C61 to C59, R50 to R48, R51 to R49, R52 to R50, U12 to U11
Changed lines of the file:
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@@
   (symbol (lib_id "power:GND") (at 99.06 110.49 0) (unit 1)
     (in_bom yes) (on_board yes)
-    (property "Reference" "#PWR0126" (id 0) (at 99.06 116.84 0)
+    (property "Reference" "#PWR0112" (id 0) (at 99.06 116.84 0)
       (effects (font (size 1.27 1.27)) hide)
     )
@@
   (symbol (lib_id "Device:C") (at 88.9 96.52 0) (unit 1)
     (in_bom yes) (on_board yes)
-    (property "Reference" "C58" (id 0) (at 91.44 95.25 0)
+    (property "Reference" "C56" (id 0) (at 91.44 95.25 0)
       (effects (font (size 1.27 1.27)) (justify left))
     )
@@
   (symbol (lib_id "Device:C") (at 99.06 96.52 0) (unit 1)
     (in_bom yes) (on_board yes)
-    (property "Reference" "C59" (id 0) (at 101.6 95.25 0)
+    (property "Reference" "C57" (id 0) (at 101.6 95.25 0)
       (effects (font (size 1.27 1.27)) (justify left))
     )
@@
   (symbol (lib_id "power:GND") (at 88.9 110.49 0) (unit 1)
     (in_bom yes) (on_board yes)
-    (property "Reference" "#PWR0125" (id 0) (at 88.9 116.84 0)
+    (property "Reference" "#PWR0111" (id 0) (at 88.9 116.84 0)
       (effects (font (size 1.27 1.27)) hide)
     )
@@
   (symbol (lib_id "power:GND") (at 109.22 110.49 0) (unit 1)
     (in_bom yes) (on_board yes)
-    (property "Reference" "#PWR0127" (id 0) (at 109.22 116.84 0)
+    (property "Reference" "#PWR0113" (id 0) (at 109.22 116.84 0)
       (effects (font (size 1.27 1.27)) hide)
     )
@@
   (symbol (lib_id "power:GND") (at 179.07 110.49 0) (unit 1)
     (in_bom yes) (on_board yes)
-    (property "Reference" "#PWR0130" (id 0) (at 179.07 116.84 0)
+    (property "Reference" "#PWR0116" (id 0) (at 179.07 116.84 0)
       (effects (font (size 1.27 1.27)) hide)
     )
@@
   (symbol (lib_id "omodri_lib:TPSM561R5") (at 140.97 87.63 0) (unit 1)
     (in_bom yes) (on_board yes)
-    (property "Reference" "U12" (id 0) (at 140.97 77.47 0))
+    (property "Reference" "U11" (id 0) (at 140.97 77.47 0))
     (property "Value" "TPSM561R5" (id 1) (at 140.97 80.01 0))
     (property "Footprint" "udriver3:B3QFN_15" (id 2) (at 140.97 87.63 0)
@@
   (symbol (lib_id "Device:C") (at 109.22 96.52 0) (unit 1)
     (in_bom yes) (on_board yes)
-    (property "Reference" "C60" (id 0) (at 111.76 95.25 0)
+    (property "Reference" "C58" (id 0) (at 111.76 95.25 0)
       (effects (font (size 1.27 1.27)) (justify left))
     )
@@
   (symbol (lib_id "Device:C") (at 187.96 96.52 0) (unit 1)
     (in_bom yes) (on_board yes)
-    (property "Reference" "C61" (id 0) (at 190.881 95.3516 0)
+    (property "Reference" "C59" (id 0) (at 190.881 95.3516 0)
       (effects (font (size 1.27 1.27)) (justify left))
     )
@@
   (symbol (lib_id "Device:R") (at 179.07 104.14 180) (unit 1)
     (in_bom yes) (on_board yes)
-    (property "Reference" "R52" (id 0) (at 184.15 102.87 0)
+    (property "Reference" "R50" (id 0) (at 184.15 102.87 0)
       (effects (font (size 1.27 1.27)) (justify left))
     )
@@
   (symbol (lib_id "power:GND") (at 124.46 110.49 0) (unit 1)
     (in_bom yes) (on_board yes)
-    (property "Reference" "#PWR0128" (id 0) (at 124.46 116.84 0)
+    (property "Reference" "#PWR0114" (id 0) (at 124.46 116.84 0)
       (effects (font (size 1.27 1.27)) hide)
     )
@@
   (symbol (lib_id "power:GND") (at 165.1 110.49 0) (unit 1)
     (in_bom yes) (on_board yes)
-    (property "Reference" "#PWR0129" (id 0) (at 165.1 116.84 0)
+    (property "Reference" "#PWR0115" (id 0) (at 165.1 116.84 0)
       (effects (font (size 1.27 1.27)) hide)
     )
@@
   (symbol (lib_id "power:GND") (at 187.96 110.49 0) (unit 1)
     (in_bom yes) (on_board yes)
-    (property "Reference" "#PWR0131" (id 0) (at 187.96 116.84 0)
+    (property "Reference" "#PWR0117" (id 0) (at 187.96 116.84 0)
       (effects (font (size 1.27 1.27)) hide)
     )
@@
   (symbol (lib_id "Device:R") (at 179.07 87.63 0) (unit 1)
     (in_bom yes) (on_board yes)
-    (property "Reference" "R50" (id 0) (at 180.848 86.4616 0)
+    (property "Reference" "R48" (id 0) (at 180.848 86.4616 0)
       (effects (font (size 1.27 1.27)) (justify left))
     )
@@
   (symbol (lib_id "Device:R") (at 165.1 99.06 0) (unit 1)
     (in_bom yes) (on_board yes)
-    (property "Reference" "R51" (id 0) (at 166.878 97.8916 0)
-      (effects (font (size 1.27 1.27)) (justify left))
-    )
+    (property "Reference" "R49" (id 0) (at 166.878 97.8916 0)
+      (effects (font (size 1.27 1.27)) (justify left))
+    )

Commit message: Repositioning of CAN resistor.
Parts:
- U11: value TPSM561R5 -> TPSM5601R5; DigiKey (none) -> 296-TPSM5601R5HSRDARTR-ND; Mouser (none) -> 595-TPSM5601R5HSRDAR; Part No (none) -> TPSM5601R5HSRDAR
Changed lines of the file:
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@@
     (in_bom yes) (on_board yes)
     (property "Reference" "U11" (id 0) (at 140.97 77.47 0))
-    (property "Value" "TPSM561R5" (id 1) (at 140.97 80.01 0))
+    (property "Value" "TPSM5601R5" (id 1) (at 140.97 80.01 0))
     (property "Footprint" "udriver3:B3QFN_15" (id 2) (at 140.97 87.63 0)
       (effects (font (size 1.27 1.27)) hide)
@@
       (effects (font (size 1.27 1.27)) hide)
     )
+    (property "DigiKey" "296-TPSM5601R5HSRDARTR-ND" (id 4) (at 140.97 87.63 0)
+      (effects (font (size 1.27 1.27)) hide)
+    )
+    (property "Mouser" "595-TPSM5601R5HSRDAR" (id 5) (at 140.97 87.63 0)
+      (effects (font (size 1.27 1.27)) hide)
+    )
+    (property "Part No" "TPSM5601R5HSRDAR" (id 6) (at 140.97 87.63 0)
+      (effects (font (size 1.27 1.27)) hide)
+    )

Commit message: Gerber update, missing ordering reference added and project BOM.
Parts:
- U11: DigiKey 296-TPSM5601R5HSRDARTR-ND -> 296-TPSM5601R5RDARTR-ND; Mouser 595-TPSM5601R5HSRDAR -> 595-TPSM5601R5SRDAR; Part No TPSM5601R5HSRDAR -> TPSM5601R5RDAR
Changed lines of the file:
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@@
       (effects (font (size 1.27 1.27)) hide)
     )
-    (property "DigiKey" "296-TPSM5601R5HSRDARTR-ND" (id 4) (at 140.97 87.63 0)
+    (property "DigiKey" "296-TPSM5601R5RDARTR-ND" (id 4) (at 140.97 87.63 0)
       (effects (font (size 1.27 1.27)) hide)
     )
-    (property "Mouser" "595-TPSM5601R5HSRDAR" (id 5) (at 140.97 87.63 0)
+    (property "Mouser" "595-TPSM5601R5SRDAR" (id 5) (at 140.97 87.63 0)
       (effects (font (size 1.27 1.27)) hide)
     )
-    (property "Part No" "TPSM5601R5HSRDAR" (id 6) (at 140.97 87.63 0)
+    (property "Part No" "TPSM5601R5RDAR" (id 6) (at 140.97 87.63 0)
       (effects (font (size 1.27 1.27)) hide)
     )
