File: hardware/udriver3/OMODRI_IMU_DBG.kicad_sch (KiCad schematic)
At the start: 6 parts, among them J1 Conn_01x10, U19 BMI088

Commit message: PCB udpates. - add serial resistors on boot jumpers - modify config jumpers to be opened by default
Parts:
- added R59, R60: 10k, Resistor_SMD:R_0201_0603Metric, symbol Device:R
- renumbered C104 to C100, C103 to C99, J1 to J12, JP1 to JP5, JP2 to JP6, U19 to U16
Connections:
- net BOOT_MODE0 renamed BOOT_0
- net BOOT_0: now also R59.1
- net DBG_GPIO0 renamed DBG_GPIO_0
- net DBG_GPIO1 renamed DBG_GPIO_1
- net DBG_GPIO2 renamed DBG_GPIO_2
- net DBG_GPIO3 renamed DBG_GPIO_3
- net ~{DBG_SPI_CSn}_BOOT_MODE1 renamed BOOT_1
- net BOOT_1: now also R60.1; no longer J12.7 (Pin_7)
- new net BOOT_MODE_0: R59.2
- new net ~{DBG_SPI_CSn}_BOOT_MODE_1: J12.7 (Pin_7), R60.2
Other:
- moved on the sheet: JP5, JP6

Commit message: PCB updates.
Parts:
- JP5, JP6: footprint Jumper:SolderJumper-3_P1.3mm_Open_Pad1.0x1.5mm_NumberLabels -> Jumper:SolderJumper-3_P2.0mm_Open_TrianglePad1.0x1.5mm
Changed lines of the file:
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@@
       (effects (font (size 1.27 1.27)) (justify left) hide)
     )
-    (property "Footprint" "Jumper:SolderJumper-3_P1.3mm_Open_Pad1.0x1.5mm_NumberLabels" (id 2) (at 82.55 55.88 0)
+    (property "Footprint" "Jumper:SolderJumper-3_P2.0mm_Open_TrianglePad1.0x1.5mm" (id 2) (at 82.55 55.88 0)
       (effects (font (size 1.27 1.27)) hide)
     )
@@
       (effects (font (size 1.27 1.27)) (justify left) hide)
     )
-    (property "Footprint" "Jumper:SolderJumper-3_P1.3mm_Open_Pad1.0x1.5mm_NumberLabels" (id 2) (at 88.9 68.58 0)
+    (property "Footprint" "Jumper:SolderJumper-3_P2.0mm_Open_TrianglePad1.0x1.5mm" (id 2) (at 88.9 68.58 0)
       (effects (font (size 1.27 1.27)) hide)
     )

Commit message: Repositioning of CAN resistor.
Parts:
- U16: DigiKey (none) -> 828-1082-2-ND; Mouser (none) -> 262-BMI088; Part No (none) -> BMI088
Changed lines of the file:
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@@
+      (effects (font (size 1.27 1.27)) hide)
+    )
+    (property "DigiKey" "828-1082-2-ND" (id 4) (at 147.32 115.57 0)
+      (effects (font (size 1.27 1.27)) hide)
+    )
+    (property "Mouser" "262-BMI088" (id 5) (at 147.32 115.57 0)
+      (effects (font (size 1.27 1.27)) hide)
+    )
+    (property "Part No" "BMI088" (id 6) (at 147.32 115.57 0)
       (effects (font (size 1.27 1.27)) hide)
     )

Commit message: Schematics updates (DC/DC description).
Parts:
- JP5, JP6: footprint Jumper:SolderJumper-3_P2.0mm_Open_TrianglePad1.0x1.5mm -> Jumper:SolderJumper-3_P2.0mm_Open_TrianglePad1.0x1.5mm_NumberLabels
Changed lines of the file:
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@@
       (effects (font (size 1.27 1.27)) (justify left) hide)
     )
-    (property "Footprint" "Jumper:SolderJumper-3_P2.0mm_Open_TrianglePad1.0x1.5mm" (id 2) (at 82.55 55.88 0)
+    (property "Footprint" "Jumper:SolderJumper-3_P2.0mm_Open_TrianglePad1.0x1.5mm_NumberLabels" (id 2) (at 82.55 55.88 0)
       (effects (font (size 1.27 1.27)) hide)
     )
@@
       (effects (font (size 1.27 1.27)) (justify left) hide)
     )
-    (property "Footprint" "Jumper:SolderJumper-3_P2.0mm_Open_TrianglePad1.0x1.5mm" (id 2) (at 88.9 68.58 0)
+    (property "Footprint" "Jumper:SolderJumper-3_P2.0mm_Open_TrianglePad1.0x1.5mm_NumberLabels" (id 2) (at 88.9 68.58 0)
       (effects (font (size 1.27 1.27)) hide)
     )

Commit message: Modify JP5/JP6 jumper to remove DRC error. Add gate resistor on power MOSFET (high & low side).
Parts:
- JP5, JP6: footprint Jumper:SolderJumper-3_P2.0mm_Open_TrianglePad1.0x1.5mm_NumberLabels -> udriver3:SolderJumper-3_P2.0mm_Open_TrianglePad1.0x1.5mm_NumberLabels
Changed lines of the file:
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@@
     (title "Open MOtor DRiver Initiative (OMODRI)")
     (date "2022-11-24")
-    (rev "2.0")
+    (rev "3.0")
     (company "LAAS/CNRS")
   )
@@
       (effects (font (size 1.27 1.27)) (justify left) hide)
     )
-    (property "Footprint" "Jumper:SolderJumper-3_P2.0mm_Open_TrianglePad1.0x1.5mm_NumberLabels" (at 82.55 55.88 0)
+    (property "Footprint" "udriver3:SolderJumper-3_P2.0mm_Open_TrianglePad1.0x1.5mm_NumberLabels" (at 82.55 55.88 0)
       (effects (font (size 1.27 1.27)) hide)
     )
@@
       (effects (font (size 1.27 1.27)) (justify left) hide)
     )
-    (property "Footprint" "Jumper:SolderJumper-3_P2.0mm_Open_TrianglePad1.0x1.5mm_NumberLabels" (at 88.9 68.58 0)
-      (effects (font (size 1.27 1.27)) hide)
-    )
+    (property "Footprint" "udriver3:SolderJumper-3_P2.0mm_Open_TrianglePad1.0x1.5mm_NumberLabels" (at 88.9 68.58 0)
+      (effects (font (size 1.27 1.27)) hide)
+    )

Commit message: update 3D models. Modify the SPI CS debug pin previously shared with boot function. Regen gerber files.
Connections:
- net ~{DBG_SPI_CSn}_BOOT_MODE_1 renamed BOOT_MODE_1
- net BOOT_MODE_1: no longer J12.7 (Pin_7)
- new net ~{DBG_SPI_CSn}: J12.7 (Pin_7)
Changed lines of the file:
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@@
     (effects (font (size 1.27 1.27)) (justify left))
   )
-  (hierarchical_label "~{DBG_SPI_CSn}_BOOT_MODE_1" (shape input) (at 182.88 67.31 180) (fields_autoplaced)
+  (hierarchical_label "~{DBG_SPI_CSn}" (shape input) (at 182.88 67.31 180) (fields_autoplaced)
     (effects (font (size 1.27 1.27)) (justify right))
   )
@@
     (effects (font (size 1.27 1.27)) (justify left))
   )
-  (hierarchical_label "~{DBG_SPI_CSn}_BOOT_MODE_1" (shape input) (at 114.3 68.58 0) (fields_autoplaced)
+  (hierarchical_label "BOOT_MODE_1" (shape passive) (at 114.3 68.58 0) (fields_autoplaced)
     (effects (font (size 1.27 1.27)) (justify left))
   )
