File: hardware/udriver3/OMODRI_ETHERCAT_CONNECT.kicad_sch (KiCad schematic)
At the start: 2 parts, among them J15 ADM6_ADF6, J16 ADM6_ADF6

Commit message: PCB update. Re-annotation of the design + via stitching (GND).
Parts:
- renumbered J16 to J11, J15 to J12
Changed lines of the file:
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@@
   (symbol (lib_id "power:GND") (at 150.495 95.25 0) (unit 1)
     (in_bom yes) (on_board yes)
-    (property "Reference" "#PWR0155" (id 0) (at 150.495 101.6 0)
+    (property "Reference" "#PWR091" (id 0) (at 150.495 101.6 0)
       (effects (font (size 1.27 1.27)) hide)
     )
@@
   (symbol (lib_id "power:GND") (at 188.595 95.25 0) (unit 1)
     (in_bom yes) (on_board yes)
-    (property "Reference" "#PWR0156" (id 0) (at 188.595 101.6 0)
+    (property "Reference" "#PWR092" (id 0) (at 188.595 101.6 0)
       (effects (font (size 1.27 1.27)) hide)
     )
@@
   (symbol (lib_id "omodri_lib:ADM6_ADF6") (at 80.01 82.55 0) (unit 1)
     (in_bom yes) (on_board yes)
-    (property "Reference" "J16" (id 0) (at 80.01 68.58 0)
+    (property "Reference" "J11" (id 0) (at 80.01 68.58 0)
       (effects (font (size 1.27 1.27)) (justify left))
     )
@@
   (symbol (lib_id "omodri_lib:ADM6_ADF6") (at 118.11 82.55 0) (unit 2)
     (in_bom yes) (on_board yes)
-    (property "Reference" "J16" (id 0) (at 118.11 68.58 0)
+    (property "Reference" "J11" (id 0) (at 118.11 68.58 0)
       (effects (font (size 1.27 1.27)) (justify left))
     )
@@
   (symbol (lib_id "omodri_lib:ADM6_ADF6") (at 158.115 82.55 0) (unit 3)
     (in_bom yes) (on_board yes)
-    (property "Reference" "J16" (id 0) (at 158.115 68.58 0)
+    (property "Reference" "J11" (id 0) (at 158.115 68.58 0)
       (effects (font (size 1.27 1.27)) (justify left))
     )
@@
   (symbol (lib_id "omodri_lib:ADM6_ADF6") (at 196.215 82.55 0) (unit 4)
     (in_bom yes) (on_board yes)
-    (property "Reference" "J16" (id 0) (at 196.215 68.58 0)
+    (property "Reference" "J11" (id 0) (at 196.215 68.58 0)
       (effects (font (size 1.27 1.27)) (justify left))
     )
@@
   (symbol (lib_id "omodri_lib:ADM6_ADF6") (at 80.01 120.65 0) (unit 1)
     (in_bom yes) (on_board yes)
-    (property "Reference" "J15" (id 0) (at 80.01 106.68 0)
+    (property "Reference" "J12" (id 0) (at 80.01 106.68 0)
       (effects (font (size 1.27 1.27)) (justify left))
     )
@@
   (symbol (lib_id "omodri_lib:ADM6_ADF6") (at 118.11 120.65 0) (unit 2)
     (in_bom yes) (on_board yes)
-    (property "Reference" "J15" (id 0) (at 118.11 106.68 0)
+    (property "Reference" "J12" (id 0) (at 118.11 106.68 0)
       (effects (font (size 1.27 1.27)) (justify left))
     )
@@
   (symbol (lib_id "omodri_lib:ADM6_ADF6") (at 158.115 120.65 0) (unit 3)
     (in_bom yes) (on_board yes)
-    (property "Reference" "J15" (id 0) (at 158.115 106.68 0)
+    (property "Reference" "J12" (id 0) (at 158.115 106.68 0)
       (effects (font (size 1.27 1.27)) (justify left))
     )
@@
   (symbol (lib_id "omodri_lib:ADM6_ADF6") (at 196.215 120.65 0) (unit 4)
     (in_bom yes) (on_board yes)
-    (property "Reference" "J15" (id 0) (at 196.215 106.68 0)
+    (property "Reference" "J12" (id 0) (at 196.215 106.68 0)
       (effects (font (size 1.27 1.27)) (justify left))
     )
@@
   (symbol (lib_id "power:GND") (at 110.49 133.35 0) (unit 1)
     (in_bom yes) (on_board yes)
-    (property "Reference" "#PWR0161" (id 0) (at 110.49 139.7 0)
+    (property "Reference" "#PWR094" (id 0) (at 110.49 139.7 0)
       (effects (font (size 1.27 1.27)) hide)
     )
@@
   (symbol (lib_id "power:GND") (at 72.39 133.35 0) (unit 1)
     (in_bom yes) (on_board yes)
-    (property "Reference" "#PWR0160" (id 0) (at 72.39 139.7 0)
-      (effects (font (size 1.27 1.27)) hide)
-    )
+    (property "Reference" "#PWR093" (id 0) (at 72.39 139.7 0)
+      (effects (font (size 1.27 1.27)) hide)
+    )

Commit message: PCB udpates. - add serial resistors on boot jumpers - modify config jumpers to be opened by default
Parts:
- renumbered J11 to J8, J12 to J9
Changed lines of the file:
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@@
   (symbol (lib_id "power:GND") (at 150.495 95.25 0) (unit 1)
     (in_bom yes) (on_board yes)
-    (property "Reference" "#PWR092" (id 0) (at 150.495 101.6 0)
+    (property "Reference" "#PWR078" (id 0) (at 150.495 101.6 0)
       (effects (font (size 1.27 1.27)) hide)
     )
@@
   (symbol (lib_id "power:GND") (at 188.595 95.25 0) (unit 1)
     (in_bom yes) (on_board yes)
-    (property "Reference" "#PWR093" (id 0) (at 188.595 101.6 0)
+    (property "Reference" "#PWR079" (id 0) (at 188.595 101.6 0)
       (effects (font (size 1.27 1.27)) hide)
     )
@@
   (symbol (lib_id "omodri_lib:ADM6_ADF6") (at 80.01 82.55 0) (unit 1)
     (in_bom yes) (on_board yes)
-    (property "Reference" "J11" (id 0) (at 80.01 68.58 0)
+    (property "Reference" "J8" (id 0) (at 80.01 68.58 0)
       (effects (font (size 1.27 1.27)) (justify left))
     )
@@
   (symbol (lib_id "omodri_lib:ADM6_ADF6") (at 118.11 82.55 0) (unit 2)
     (in_bom yes) (on_board yes)
-    (property "Reference" "J11" (id 0) (at 118.11 68.58 0)
+    (property "Reference" "J8" (id 0) (at 118.11 68.58 0)
       (effects (font (size 1.27 1.27)) (justify left))
     )
@@
   (symbol (lib_id "omodri_lib:ADM6_ADF6") (at 158.115 82.55 0) (unit 3)
     (in_bom yes) (on_board yes)
-    (property "Reference" "J11" (id 0) (at 158.115 68.58 0)
+    (property "Reference" "J8" (id 0) (at 158.115 68.58 0)
       (effects (font (size 1.27 1.27)) (justify left))
     )
@@
   (symbol (lib_id "omodri_lib:ADM6_ADF6") (at 196.215 82.55 0) (unit 4)
     (in_bom yes) (on_board yes)
-    (property "Reference" "J11" (id 0) (at 196.215 68.58 0)
+    (property "Reference" "J8" (id 0) (at 196.215 68.58 0)
       (effects (font (size 1.27 1.27)) (justify left))
     )
@@
   (symbol (lib_id "omodri_lib:ADM6_ADF6") (at 80.01 120.65 0) (unit 1)
     (in_bom yes) (on_board yes)
-    (property "Reference" "J12" (id 0) (at 80.01 106.68 0)
+    (property "Reference" "J9" (id 0) (at 80.01 106.68 0)
       (effects (font (size 1.27 1.27)) (justify left))
     )
@@
   (symbol (lib_id "omodri_lib:ADM6_ADF6") (at 118.11 120.65 0) (unit 2)
     (in_bom yes) (on_board yes)
-    (property "Reference" "J12" (id 0) (at 118.11 106.68 0)
+    (property "Reference" "J9" (id 0) (at 118.11 106.68 0)
       (effects (font (size 1.27 1.27)) (justify left))
     )
@@
   (symbol (lib_id "omodri_lib:ADM6_ADF6") (at 158.115 120.65 0) (unit 3)
     (in_bom yes) (on_board yes)
-    (property "Reference" "J12" (id 0) (at 158.115 106.68 0)
+    (property "Reference" "J9" (id 0) (at 158.115 106.68 0)
       (effects (font (size 1.27 1.27)) (justify left))
     )
@@
   (symbol (lib_id "omodri_lib:ADM6_ADF6") (at 196.215 120.65 0) (unit 4)
     (in_bom yes) (on_board yes)
-    (property "Reference" "J12" (id 0) (at 196.215 106.68 0)
+    (property "Reference" "J9" (id 0) (at 196.215 106.68 0)
       (effects (font (size 1.27 1.27)) (justify left))
     )
@@
   (symbol (lib_id "power:GND") (at 110.49 133.35 0) (unit 1)
     (in_bom yes) (on_board yes)
-    (property "Reference" "#PWR095" (id 0) (at 110.49 139.7 0)
+    (property "Reference" "#PWR081" (id 0) (at 110.49 139.7 0)
       (effects (font (size 1.27 1.27)) hide)
     )
@@
   (symbol (lib_id "power:GND") (at 72.39 133.35 0) (unit 1)
     (in_bom yes) (on_board yes)
-    (property "Reference" "#PWR094" (id 0) (at 72.39 139.7 0)
-      (effects (font (size 1.27 1.27)) hide)
-    )
+    (property "Reference" "#PWR080" (id 0) (at 72.39 139.7 0)
+      (effects (font (size 1.27 1.27)) hide)
+    )

Commit message: Add JLCPCB components ref where it was matching.
Parts:
- J8, J9: LCSC (none) -> C3645391
Changed lines of the file:
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@@
+      (effects (font (size 1.27 1.27)) hide)
+    )
+    (property "LCSC" "C3645391" (at 80.01 82.55 0)
       (effects (font (size 1.27 1.27)) hide)
     )
@@
       (effects (font (size 1.27 1.27)) hide)
     )
+    (property "LCSC" "C3645391" (at 118.11 82.55 0)
+      (effects (font (size 1.27 1.27)) hide)
+    )
     (pin "A01")
     (pin "A02")
@@
       (effects (font (size 1.27 1.27)) hide)
     )
+    (property "LCSC" "C3645391" (at 158.115 82.55 0)
+      (effects (font (size 1.27 1.27)) hide)
+    )
     (pin "A01")
     (pin "A02")
@@
       (effects (font (size 1.27 1.27)) hide)
     )
+    (property "LCSC" "C3645391" (at 196.215 82.55 0)
+      (effects (font (size 1.27 1.27)) hide)
+    )
     (pin "A01")
     (pin "A02")
@@
       (effects (font (size 1.27 1.27)) hide)
     )
+    (property "LCSC" "C3645391" (at 80.01 120.65 0)
+      (effects (font (size 1.27 1.27)) hide)
+    )
     (pin "A01")
     (pin "A02")
@@
       (effects (font (size 1.27 1.27)) hide)
     )
+    (property "LCSC" "C3645391" (at 118.11 120.65 0)
+      (effects (font (size 1.27 1.27)) hide)
+    )
     (pin "A01")
     (pin "A02")
@@
       (effects (font (size 1.27 1.27)) hide)
     )
+    (property "LCSC" "C3645391" (at 158.115 120.65 0)
+      (effects (font (size 1.27 1.27)) hide)
+    )
     (pin "A01")
     (pin "A02")
@@
       (effects (font (size 1.27 1.27)) hide)
     )
+    (property "LCSC" "C3645391" (at 196.215 120.65 0)
+      (effects (font (size 1.27 1.27)) hide)
+    )
