File: hardware/udriver3_sa/OMODRI_Alim_5V.kicad_sch (KiCad schematic)
At the start: 10 parts, among them U12 TPSM8290x

Commit message: Third release of uOmodri Single Axis (uOmodri_SA). Add Test points.
Parts:
- added TP7: TestPoint, TestPoint:TestPoint_Pad_D1.0mm, symbol Connector:TestPoint
Connections:
- net 5V0: now also TP7.1
Changed lines of the file:
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@@
+	)
+	(symbol
+		(lib_id "Connector:TestPoint")
+		(at 222.25 86.36 0)
+		(unit 1)
+		(exclude_from_sim no)
+		(in_bom no)
+		(on_board yes)
+		(dnp no)
+		(fields_autoplaced yes)
+		(property "Reference" "TP7"
+			(at 224.79 81.7879 0)
+			(effects
+				(font
+					(size 1.27 1.27)
+				)
+				(justify left)
+			)
+		)
+		(property "Value" "TestPoint"
+			(at 224.79 84.3279 0)
+			(effects
+				(font
+					(size 1.27 1.27)
+				)
+				(justify left)
+			)
+		)
+		(property "Footprint" "TestPoint:TestPoint_Pad_D1.0mm"
+			(at 227.33 86.36 0)
+			(effects
+				(font
+					(size 1.27 1.27)
+				)
+				(hide yes)
+			)
+		)
+		(property "Datasheet" "~"
+			(at 227.33 86.36 0)
+			(effects
+				(font
+					(size 1.27 1.27)
+				)
+				(hide yes)
+			)
+		)
+		(property "Description" "test point"
+			(at 222.25 86.36 0)
+			(effects
+				(font
+					(size 1.27 1.27)
+				)
+				(hide yes)
+			)
+		)
+		(pin "1"
+		)
+		(instances
+			(project "omodri_sa_laas"
+				(path "/de5b13f0-933a-4c4d-9979-13dc57b13241/00000000-0000-0000-0000-00005f3a3f16/00000000-0000-0000-0000-00005f5bd908"
+					(reference "TP7")
+					(unit 1)
+				)
+			)
+		)
 	)
 	(symbol

Commit message: Update on uOmodri_SA. Remove USB, com SPI & debug connectors for integration into Myactuator motors. Connectors replaced by a ZIF connector.
Parts:
- renumbered C93 to C92, C94 to C93, C95 to C94, C96 to C95, C97 to C96, C98 to C97, R45 to R43, R46 to R44, R47 to R45, TP7 to TP4
Changed lines of the file:
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@@
 	(title_block
 		(title "Open MOtor DRiver Initiative  - Single Axis (OMODRI_SA)")
-		(date "2024-03-20")
+		(date "2024-11-08")
 		(rev "1.0")
 		(company "LAAS/CNRS")
@@
 		(on_board yes)
 		(dnp no)
-		(property "Reference" "C94"
+		(property "Reference" "C93"
 			(at 199.771 106.7816 0)
 			(effects
@@
 			(project "omodri_sa_laas"
 				(path "/de5b13f0-933a-4c4d-9979-13dc57b13241/00000000-0000-0000-0000-00005f3a3f16/00000000-0000-0000-0000-00005f5bd908"
-					(reference "C94")
+					(reference "C93")
 					(unit 1)
 				)
@@
 		(on_board yes)
 		(dnp no)
-		(property "Reference" "#PWR0156"
+		(property "Reference" "#PWR0141"
 			(at 234.95 133.35 0)
 			(effects
@@
 			(project "omodri_sa_laas"
 				(path "/de5b13f0-933a-4c4d-9979-13dc57b13241/00000000-0000-0000-0000-00005f3a3f16/00000000-0000-0000-0000-00005f5bd908"
-					(reference "#PWR0156")
+					(reference "#PWR0141")
 					(unit 1)
 				)
@@
 		(on_board yes)
 		(dnp no)
-		(property "Reference" "C95"
+		(property "Reference" "C94"
 			(at 212.471 106.7816 0)
 			(effects
@@
 			(project "omodri_sa_laas"
 				(path "/de5b13f0-933a-4c4d-9979-13dc57b13241/00000000-0000-0000-0000-00005f3a3f16/00000000-0000-0000-0000-00005f5bd908"
-					(reference "C95")
+					(reference "C94")
 					(unit 1)
 				)
@@
 		(on_board yes)
 		(dnp no)
-		(property "Reference" "#PWR0152"
+		(property "Reference" "#PWR0137"
 			(at 184.15 133.35 0)
 			(effects
@@
 			(project "omodri_sa_laas"
 				(path "/de5b13f0-933a-4c4d-9979-13dc57b13241/00000000-0000-0000-0000-00005f3a3f16/00000000-0000-0000-0000-00005f5bd908"
-					(reference "#PWR0152")
+					(reference "#PWR0137")
 					(unit 1)
 				)
@@
 		(dnp no)
 		(fields_autoplaced yes)
-		(property "Reference" "TP7"
+		(property "Reference" "TP4"
 			(at 224.79 81.7879 0)
 			(effects
@@
 			(project "omodri_sa_laas"
 				(path "/de5b13f0-933a-4c4d-9979-13dc57b13241/00000000-0000-0000-0000-00005f3a3f16/00000000-0000-0000-0000-00005f5bd908"
-					(reference "TP7")
+					(reference "TP4")
 					(unit 1)
 				)
@@
 		(on_board yes)
 		(dnp no)
-		(property "Reference" "#PWR0154"
+		(property "Reference" "#PWR0139"
 			(at 209.55 133.35 0)
 			(effects
@@
 			(project "omodri_sa_laas"
 				(path "/de5b13f0-933a-4c4d-9979-13dc57b13241/00000000-0000-0000-0000-00005f3a3f16/00000000-0000-0000-0000-00005f5bd908"
-					(reference "#PWR0154")
+					(reference "#PWR0139")
 					(unit 1)
 				)
@@
 		(on_board yes)
 		(dnp no)
-		(property "Reference" "#PWR0149"
+		(property "Reference" "#PWR0134"
 			(at 114.3 133.35 0)
 			(effects
@@
 			(project "omodri_sa_laas"
 				(path "/de5b13f0-933a-4c4d-9979-13dc57b13241/00000000-0000-0000-0000-00005f3a3f16/00000000-0000-0000-0000-00005f5bd908"
-					(reference "#PWR0149")
+					(reference "#PWR0134")
 					(unit 1)
 				)
@@
 		(on_board yes)
 		(dnp no)
-		(property "Reference" "C97"
+		(property "Reference" "C96"
 			(at 237.871 106.7816 0)
 			(effects
@@
 			(project "omodri_sa_laas"
 				(path "/de5b13f0-933a-4c4d-9979-13dc57b13241/00000000-0000-0000-0000-00005f3a3f16/00000000-0000-0000-0000-00005f5bd908"
-					(reference "C97")
+					(reference "C96")
 					(unit 1)
 				)
@@
 		(on_board yes)
 		(dnp no)
-		(property "Reference" "C98"
+		(property "Reference" "C97"
 			(at 127.635 118.11 0)
 			(effects
@@
 			(project "omodri_sa_laas"
 				(path "/de5b13f0-933a-4c4d-9979-13dc57b13241/00000000-0000-0000-0000-00005f3a3f16/00000000-0000-0000-0000-00005f5bd908"
-					(reference "C98")
+					(reference "C97")
 					(unit 1)
 				)
@@
 		(on_board yes)
 		(dnp no)
-		(property "Reference" "R47"
+		(property "Reference" "R45"
 			(at 189.23 106.68 0)
 			(effects
@@
 			(project "omodri_sa_laas"
 				(path "/de5b13f0-933a-4c4d-9979-13dc57b13241/00000000-0000-0000-0000-00005f3a3f16/00000000-0000-0000-0000-00005f5bd908"
-					(reference "R47")
+					(reference "R45")
 					(unit 1)
 				)
@@
 		(on_board yes)
 		(dnp no)
-		(property "Reference" "#PWR0151"
+		(property "Reference" "#PWR0136"
 			(at 165.1 133.35 0)
 			(effects
@@
 			(project "omodri_sa_laas"
 				(path "/de5b13f0-933a-4c4d-9979-13dc57b13241/00000000-0000-0000-0000-00005f3a3f16/00000000-0000-0000-0000-00005f5bd908"
-					(reference "#PWR0151")
+					(reference "#PWR0136")
 					(unit 1)
 				)
@@
 		(on_board yes)
 		(dnp no)
-		(property "Reference" "R45"
+		(property "Reference" "R43"
 			(at 173.228 90.2716 0)
 			(effects
@@
 			(project "omodri_sa_laas"
 				(path "/de5b13f0-933a-4c4d-9979-13dc57b13241/00000000-0000-0000-0000-00005f3a3f16/00000000-0000-0000-0000-00005f5bd908"
-					(reference "R45")
+					(reference "R43")
 					(unit 1)
 				)
@@
 		(on_board yes)
 		(dnp no)
-		(property "Reference" "C96"
+		(property "Reference" "C95"
 			(at 225.171 106.7816 0)
 			(effects
@@
 			(project "omodri_sa_laas"
 				(path "/de5b13f0-933a-4c4d-9979-13dc57b13241/00000000-0000-0000-0000-00005f3a3f16/00000000-0000-0000-0000-00005f5bd908"
-					(reference "C96")
+					(reference "C95")
 					(unit 1)
 				)
@@
 		(on_board yes)
 		(dnp no)
-		(property "Reference" "R46"
+		(property "Reference" "R44"
 			(at 185.928 90.2716 0)
 			(effects
@@
 			(project "omodri_sa_laas"
 				(path "/de5b13f0-933a-4c4d-9979-13dc57b13241/00000000-0000-0000-0000-00005f3a3f16/00000000-0000-0000-0000-00005f5bd908"
-					(reference "R46")
+					(reference "R44")
 					(unit 1)
 				)
@@
 		(on_board yes)
 		(dnp no)
-		(property "Reference" "C93"
+		(property "Reference" "C92"
 			(at 116.84 106.68 0)
 			(effects
@@
 			(project "omodri_sa_laas"
 				(path "/de5b13f0-933a-4c4d-9979-13dc57b13241/00000000-0000-0000-0000-00005f3a3f16/00000000-0000-0000-0000-00005f5bd908"
-					(reference "C93")
+					(reference "C92")
 					(unit 1)
 				)
@@
 		(on_board yes)
 		(dnp no)
-		(property "Reference" "#PWR0150"
+		(property "Reference" "#PWR0135"
 			(at 127 133.35 0)
 			(effects
@@
 			(project "omodri_sa_laas"
 				(path "/de5b13f0-933a-4c4d-9979-13dc57b13241/00000000-0000-0000-0000-00005f3a3f16/00000000-0000-0000-0000-00005f5bd908"
-					(reference "#PWR0150")
+					(reference "#PWR0135")
 					(unit 1)
 				)
@@
 		(on_board yes)
 		(dnp no)
-		(property "Reference" "#PWR0153"
+		(property "Reference" "#PWR0138"
 			(at 196.85 133.35 0)
 			(effects
@@
 			(project "omodri_sa_laas"
 				(path "/de5b13f0-933a-4c4d-9979-13dc57b13241/00000000-0000-0000-0000-00005f3a3f16/00000000-0000-0000-0000-00005f5bd908"
-					(reference "#PWR0153")
+					(reference "#PWR0138")
 					(unit 1)
 				)
@@
 		(on_board yes)
 		(dnp no)
-		(property "Reference" "#PWR0155"
+		(property "Reference" "#PWR0140"
 			(at 222.25 133.35 0)
 			(effects
@@
 			(project "omodri_sa_laas"
 				(path "/de5b13f0-933a-4c4d-9979-13dc57b13241/00000000-0000-0000-0000-00005f3a3f16/00000000-0000-0000-0000-00005f5bd908"
-					(reference "#PWR0155")
+					(reference "#PWR0140")
 					(unit 1)
 				)
