File: hardware/udriver3_sa/OMODRI_driver_M1.kicad_sch (KiCad schematic)
At the start: 34 parts, among them Q1 CSD88599Q5DC, Q2 CSD88599Q5DC, Q3 CSD88599Q5DC, U2 DRV8353S

Commit message: Update on uOmodri_SA. Remove USB, com SPI & debug connectors for integration into Myactuator motors. Connectors replaced by a ZIF connector.
Parts:
- renumbered C44 to C45, C45 to C46, C46 to C47, C47 to C48, C48 to C49, C49 to C50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
