File: hardware/udriver3_sa/OMODRI_mcu.kicad_sch (KiCad schematic)
At the start: 2 parts

Commit message: Replace the TCAN330G (5Mbps) by TCAN3414 (8Mbps) on both designs.
Other:
- sheet OMODRI_SA_GPIO ports: added none; removed GPIO_SELECT_2, GPIO_SELECT_3

Commit message: Update on uOmodri_SA. Remove USB, com SPI & debug connectors for integration into Myactuator motors. Connectors replaced by a ZIF connector.
Parts:
- renumbered R6 to R10, R7 to R11
Changed lines of the file:
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@@
 	(title_block
 		(title "Open MOtor DRiver Initiative  - Single Axis (OMODRI_SA)")
-		(date "2024-03-20")
+		(date "2024-11-08")
 		(rev "1.0")
 		(company "LAAS/CNRS")
@@
 		(on_board yes)
 		(dnp no)
-		(property "Reference" "R7"
+		(property "Reference" "R11"
 			(at 90.932 65.532 90)
 			(effects
@@
 			(project "omodri_sa_laas"
 				(path "/de5b13f0-933a-4c4d-9979-13dc57b13241/3df2ca62-85b2-4979-b739-c6d2bcf6d697"
-					(reference "R7")
+					(reference "R11")
 					(unit 1)
 				)
@@
 		(on_board yes)
 		(dnp no)
-		(property "Reference" "R6"
+		(property "Reference" "R10"
 			(at 90.678 59.182 90)
 			(effects
@@
 			(project "omodri_sa_laas"
 				(path "/de5b13f0-933a-4c4d-9979-13dc57b13241/3df2ca62-85b2-4979-b739-c6d2bcf6d697"
-					(reference "R6")
+					(reference "R10")
 					(unit 1)
 				)
