File: hardware/udriver3_sa/OMODRI_mcu_ctrl.kicad_sch (KiCad schematic)
At the start: 2 parts, among them U1 TMS320F28388D

Commit message: Update on uOmodri_SA. Remove USB, com SPI & debug connectors for integration into Myactuator motors. Connectors replaced by a ZIF connector.
Parts:
- renumbered R8 to R12
Changed lines of the file:
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@@
 	(title_block
 		(title "Open MOtor DRiver Initiative  - Single Axis (OMODRI_SA)")
-		(date "2024-03-20")
+		(date "2024-11-08")
 		(rev "1.0")
 		(company "LAAS/CNRS")
@@
 		(on_board yes)
 		(dnp no)
-		(property "Reference" "R8"
+		(property "Reference" "R12"
 			(at 173.355 78.74 90)
 			(effects
@@
 			(project "omodri_sa_laas"
 				(path "/de5b13f0-933a-4c4d-9979-13dc57b13241/3df2ca62-85b2-4979-b739-c6d2bcf6d697/086ff298-7762-4a18-be53-a5f29df3df5e"
-					(reference "R8")
+					(reference "R12")
 					(unit 1)
 				)
@@
 		(on_board yes)
 		(dnp no)
-		(property "Reference" "#PWR020"
+		(property "Reference" "#PWR017"
 			(at 184.15 83.82 0)
 			(effects
@@
 			(project "omodri_sa_laas"
 				(path "/de5b13f0-933a-4c4d-9979-13dc57b13241/3df2ca62-85b2-4979-b739-c6d2bcf6d697/086ff298-7762-4a18-be53-a5f29df3df5e"
-					(reference "#PWR020")
+					(reference "#PWR017")
 					(unit 1)
 				)
