File: hardware/udriver3_sa_v2/OMODRI_CAN_RS845.kicad_sch (KiCad schematic)
At the start: 9 parts, among them U4 TCAN3414, U5 TS3USB221E, U6 THVD2450

Commit message: Partial update of uOmodri Single Axis V2.
Parts:
- U4: LCSC (none) -> C24836183
Changed lines of the file:
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@@
 			)
 		)
-		(property "LCSC" ""
+		(property "LCSC" "C24836183"
 			(at 101.6 63.5 0)
 			(effects
