File: hardware/udriver3_sa_v2/OMODRI_Reset.kicad_sch (KiCad schematic)
At the start: 8 parts, among them Q4 NX7002BKM, SW1 B3U-1000P-B, U10 TPS3703-1.2, U9 TPS3703-3.3

Commit message: Partial update of uOmodri Single Axis V2.
Parts:
- D6: value LED GREEN -> LED AMBER; DigiKey 516-3066-1-ND -> 516-HSMA-C280CT-ND; Farnell 2494322 -> 2494320; LCSC C7466700 -> C5762821; Mouser 630-HSMG-C280 -> 630-HSMA-C280; Part No HSMG-C280 -> HSMA-C280; RS 867-6560 -> 230-5356
- R37: value 120 -> 150; DigiKey P122692CT-ND -> P122742CT-ND; Farnell 2396857 -> 2302313; LCSC C278569 -> C2074059; Mouser 667-ERJ-1GNF1200C -> 667-ERJ-1GNF1500C; Part No ERJ1GNF1200C -> ERJ1GNF1500C
Changed lines of the file:
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@@
 			)
 		)
-		(property "Value" "120"
+		(property "Value" "150"
 			(at 179.578 109.093 0)
 			(effects
@@
 			)
 		)
-		(property "Description" "0201,120Ω, 0.05W, ±1%, SMD  resistor"
-			(at 177.8 107.95 0)
-			(effects
-				(font
-					(size 1.27 1.27)
-				)
-				(hide yes)
-			)
-		)
-		(property "DigiKey" "P122692CT-ND"
-			(at 177.8 107.95 0)
-			(effects
-				(font
-					(size 1.27 1.27)
-				)
-				(hide yes)
-			)
-		)
-		(property "Farnell" "2396857"
-			(at 177.8 107.95 0)
-			(effects
-				(font
-					(size 1.27 1.27)
-				)
-				(hide yes)
-			)
-		)
-		(property "Mouser" "667-ERJ-1GNF1200C"
-			(at 177.8 107.95 0)
-			(effects
-				(font
-					(size 1.27 1.27)
-				)
-				(hide yes)
-			)
-		)
-		(property "Part No" "ERJ1GNF1200C"
+		(property "Description" "0201,150Ω, 0.05W, ±1%, SMD  resistor"
+			(at 177.8 107.95 0)
+			(effects
+				(font
+					(size 1.27 1.27)
+				)
+				(hide yes)
+			)
+		)
+		(property "DigiKey" "P122742CT-ND"
+			(at 177.8 107.95 0)
+			(effects
+				(font
+					(size 1.27 1.27)
+				)
+				(hide yes)
+			)
+		)
+		(property "Farnell" "2302313"
+			(at 177.8 107.95 0)
+			(effects
+				(font
+					(size 1.27 1.27)
+				)
+				(hide yes)
+			)
+		)
+		(property "Mouser" "667-ERJ-1GNF1500C"
+			(at 177.8 107.95 0)
+			(effects
+				(font
+					(size 1.27 1.27)
+				)
+				(hide yes)
+			)
+		)
+		(property "Part No" "ERJ1GNF1500C"
 			(at 177.8 107.95 0)
 			(effects
@@
 			)
 		)
-		(property "LCSC" "C278569"
+		(property "LCSC" "C2074059"
 			(at 177.8 107.95 0)
 			(effects
@@
 			)
 		)
-		(property "Value" "LED GREEN"
+		(property "Value" "LED AMBER"
 			(at 184.15 92.71 90)
 			(effects
@@
 			)
 		)
-		(property "Description" "0402, Top Mount miniature ChipLED, GREEN, Vf = 2.2-V @ 10-mA"
-			(at 177.8 95.25 0)
-			(effects
-				(font
-					(size 1.27 1.27)
-				)
-				(hide yes)
-			)
-		)
-		(property "DigiKey" "516-3066-1-ND"
-			(at 177.8 95.25 0)
-			(effects
-				(font
-					(size 1.27 1.27)
-				)
-				(hide yes)
-			)
-		)
-		(property "Mouser" "630-HSMG-C280"
-			(at 177.8 95.25 0)
-			(effects
-				(font
-					(size 1.27 1.27)
-				)
-				(hide yes)
-			)
-		)
-		(property "Farnell" "2494322"
-			(at 177.8 95.25 0)
-			(effects
-				(font
-					(size 1.27 1.27)
-				)
-				(hide yes)
-			)
-		)
-		(property "Part No" "HSMG-C280"
-			(at 177.8 95.25 0)
-			(effects
-				(font
-					(size 1.27 1.27)
-				)
-				(hide yes)
-			)
-		)
-		(property "RS" "867-6560"
-			(at 177.8 95.25 0)
-			(effects
-				(font
-					(size 1.27 1.27)
-				)
-				(hide yes)
-			)
-		)
-		(property "LCSC" " C7466700"
-			(at 177.8 95.25 0)
-			(effects
+		(property "Description" "0402, Top Mount miniature ChipLED, AMBER, Vf = 1.9-V @ 10-mA"
+			(at 177.8 95.25 0)
+			(effects
+				(font
+					(size 1.27 1.27)
+				)
+				(hide yes)
+			)
+		)
+		(property "DigiKey" "516-HSMA-C280CT-ND"
+			(at 177.8 95.25 0)
+			(effects
+				(font
+					(size 1.27 1.27)
+				)
+				(hide yes)
+			)
+		)
+		(property "Mouser" "630-HSMA-C280"
+			(at 177.8 95.25 0)
+			(effects
+				(font
+					(size 1.27 1.27)
+				)
+				(hide yes)
+			)
+		)
+		(property "Farnell" "2494320"
+			(at 177.8 95.25 0)
+			(effects
+				(font
+					(size 1.27 1.27)
+				)
+				(hide yes)
+			)
+		)
+		(property "Part No" "HSMA-C280"
+			(at 177.8 95.25 0)
+			(effects
+				(font
+					(size 1.27 1.27)
+				)
+				(hide yes)
+			)
+		)
+		(property "RS" "230-5356"
+			(at 177.8 95.25 0)
+			(effects
+				(font
+					(size 1.27 1.27)
+				)
+				(hide yes)
+			)
+		)
+		(property "LCSC" "C5762821"
+			(at 177.8 95.25 0)
+			(effects
