File: hardware/udriver3_sa_v2/omodri_sa_v2_laas.kicad_sch (KiCad schematic)
At the start: 21 parts, among them J1 Conn_01x11, J2 conn_01x20_MountingPins

Commit message: Udriver3 Single Axis V2. Update on RS485 communication (add McBSP + CLB).
Other:
- sheet OMODRI_SA_MCU ports: added SCI_TX_CLB_McBSP_TX; removed SCI_TX
Changed lines of the file:
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@@
 	(wire
 		(pts
-			(xy 63.5 72.39) (xy 76.2 72.39)
-		)
-		(stroke
-			(width 0)
-			(type default)
-		)
-	)
-	(wire
-		(pts
 			(xy 54.61 109.22) (xy 76.2 109.22)
 		)
@@
 	(wire
 		(pts
+			(xy 63.5 72.39) (xy 76.2 72.39)
+		)
+		(stroke
+			(width 0)
+			(type default)
+		)
+	)
+	(wire
+		(pts
 			(xy 127 93.98) (xy 139.7 93.98)
 		)
@@
 			)
 		)
-		(pin "SCI_TX" output
-			(at 76.2 72.39 180)
-			(effects
-				(font
-					(size 1.27 1.27)
-				)
-				(justify left)
-			)
-		)
 		(pin "PWM3_CHA" output
 			(at 127 48.26 0)
@@
 			(effects
 				(font
+					(size 1.27 1.27)
+				)
+				(justify left)
+			)
+		)
+		(pin "SCI_TX_CLB_McBSP_TX" output
+			(at 76.2 72.39 180)
+			(effects
+				(font
